File: src/hardware/pcb/ample/kicad/output.kicad_sch (KiCad schematic)
At the start: 1 part, among them U6 RC4580

Commit message: rev 00.01 schematics almost done
Other:
- moved on the sheet: U6A, U6C
Changed lines of the file:
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@@
 (kicad_sch (version 20230121) (generator eeschema)
   (paper "A4")
-  (hierarchical_label "AOUTA1+" (shape input) (at 71.12 73.66 180) (fields_autoplaced)
+  (hierarchical_label "AOUTA1+" (shape input) (at 76.2 67.31 180) (fields_autoplaced)
     (effects (font (size 1.27 1.27)) (justify right))
   )
-  (hierarchical_label "AOUTB1+" (shape input) (at 71.12 80.01 180) (fields_autoplaced)
+  (hierarchical_label "FILT_RIGHT" (shape output) (at 219.71 68.58 0) (fields_autoplaced)
+    (effects (font (size 1.27 1.27)) (justify left))
+  )
+  (hierarchical_label "AOUTB1+" (shape input) (at 76.2 73.66 180) (fields_autoplaced)
     (effects (font (size 1.27 1.27)) (justify right))
   )
-  (hierarchical_label "AOUTB1-" (shape input) (at 71.12 82.55 180) (fields_autoplaced)
+  (hierarchical_label "FILT_LEFT" (shape output) (at 219.71 64.77 0) (fields_autoplaced)
+    (effects (font (size 1.27 1.27)) (justify left))
+  )
+  (hierarchical_label "AOUTB1-" (shape input) (at 76.2 76.2 180) (fields_autoplaced)
     (effects (font (size 1.27 1.27)) (justify right))
   )
-  (hierarchical_label "AOUTA1-" (shape input) (at 71.12 76.2 180) (fields_autoplaced)
+  (hierarchical_label "AOUTA1-" (shape input) (at 76.2 69.85 180) (fields_autoplaced)
     (effects (font (size 1.27 1.27)) (justify right))
   )
-  (symbol (lib_id "power:GND") (at 163.83 95.25 0) (unit 1)
+  (symbol (lib_id "power:GND") (at 157.48 78.74 0) (unit 1)
     (in_bom yes) (on_board yes) (dnp no)
-    (property "Reference" "#PWR052" (at 163.83 101.6 0)
+    (property "Reference" "#PWR052" (at 157.48 85.09 0)
       (effects (font (size 1.27 1.27)) hide)
     )
-    (property "Value" "GND" (at 163.957 99.6442 0)
+    (property "Value" "GND" (at 157.607 83.1342 0)
       (effects (font (size 1.27 1.27)))
     )
-    (property "Footprint" "" (at 163.83 95.25 0)
+    (property "Footprint" "" (at 157.48 78.74 0)
       (effects (font (size 1.27 1.27)) hide)
     )
-    (property "Datasheet" "" (at 163.83 95.25 0)
+    (property "Datasheet" "" (at 157.48 78.74 0)
       (effects (font (size 1.27 1.27)) hide)
     )
@@
     )
   )
-  (symbol (lib_id "Amplifier_Operational:RC4580") (at 135.89 93.98 0) (unit 3)
+  (symbol (lib_id "Amplifier_Operational:RC4580") (at 129.54 77.47 0) (unit 3)
     (in_bom yes) (on_board yes) (dnp no) (fields_autoplaced)
-    (property "Reference" "U6" (at 134.62 92.71 0)
+    (property "Reference" "U6" (at 128.27 76.2 0)
       (effects (font (size 1.27 1.27)) (justify left))
     )
-    (property "Value" "RC4580" (at 134.62 95.25 0)
+    (property "Value" "RC4580" (at 128.27 78.74 0)
       (effects (font (size 1.27 1.27)) (justify left))
     )
-    (property "Footprint" "" (at 135.89 93.98 0)
+    (property "Footprint" "" (at 129.54 77.47 0)
       (effects (font (size 1.27 1.27)) hide)
     )
-    (property "Datasheet" "http://www.ti.com/lit/ds/symlink/rc4580.pdf" (at 135.89 93.98 0)
+    (property "Datasheet" "http://www.ti.com/lit/ds/symlink/rc4580.pdf" (at 129.54 77.47 0)
       (effects (font (size 1.27 1.27)) hide)
     )
@@
     )
   )
-  (symbol (lib_id "Amplifier_Operational:RC4580") (at 130.81 82.55 0) (unit 1)
+  (symbol (lib_id "Amplifier_Operational:RC4580") (at 124.46 66.04 0) (unit 1)
     (in_bom yes) (on_board yes) (dnp no) (fields_autoplaced)
-    (property "Reference" "U6" (at 130.81 72.39 0)
+    (property "Reference" "U6" (at 124.46 55.88 0)
       (effects (font (size 1.27 1.27)))
     )
-    (property "Value" "RC4580" (at 130.81 74.93 0)
+    (property "Value" "RC4580" (at 124.46 58.42 0)
       (effects (font (size 1.27 1.27)))
     )
-    (property "Footprint" "" (at 130.81 82.55 0)
+    (property "Footprint" "" (at 124.46 66.04 0)
       (effects (font (size 1.27 1.27)) hide)
     )
-    (property "Datasheet" "http://www.ti.com/lit/ds/symlink/rc4580.pdf" (at 130.81 82.55 0)
+    (property "Datasheet" "http://www.ti.com/lit/ds/symlink/rc4580.pdf" (at 124.46 66.04 0)
       (effects (font (size 1.27 1.27)) hide)
     )
@@
     )
   )
-  (symbol (lib_id "Amplifier_Operational:RC4580") (at 151.13 82.55 0) (unit 2)
+  (symbol (lib_id "Amplifier_Operational:RC4580") (at 124.46 99.06 0) (unit 2)
     (in_bom yes) (on_board yes) (dnp no) (fields_autoplaced)
-    (property "Reference" "U6" (at 151.13 72.39 0)
+    (property "Reference" "U6" (at 124.46 88.9 0)
       (effects (font (size 1.27 1.27)) hide)
     )
-    (property "Value" "RC4580" (at 151.13 74.93 0)
+    (property "Value" "RC4580" (at 124.46 91.44 0)
       (effects (font (size 1.27 1.27)))
     )
-    (property "Footprint" "" (at 151.13 82.55 0)
+    (property "Footprint" "" (at 124.46 99.06 0)
       (effects (font (size 1.27 1.27)) hide)
     )
-    (property "Datasheet" "http://www.ti.com/lit/ds/symlink/rc4580.pdf" (at 151.13 82.55 0)
+    (property "Datasheet" "http://www.ti.com/lit/ds/symlink/rc4580.pdf" (at 124.46 99.06 0)
       (effects (font (size 1.27 1.27)) hide)
     )
