File: src/hardware/pcb/ample/kicad/ample.kicad_pcb (KiCad board)
At the start: 2 copper layers, 54 x 80 mm, 22 parts, among them U11 CS42528, U3 MAX660MX, U5 MAX13331, U7 TORX1350A(F)

Commit message: finishing schematics
Parts:
- added C1: 10u, Capacitor_SMD:C_0603_1608Metric, F.Cu at (-7.29, -76.4)
- added C10: 100n, Capacitor_SMD:C_0603_1608Metric, F.Cu at (-7.29, -56.4)
- added C11: 10u, Capacitor_SMD:C_0603_1608Metric, F.Cu at (-7.29, -53.8)
- added C12: 10u, Capacitor_SMD:C_0603_1608Metric, F.Cu at (-7.29, -51.3)
- added C13: 2u2, Capacitor_SMD:C_0603_1608Metric, F.Cu at (-3.28, -76.4)
- added C14: 10u, Capacitor_SMD:C_0603_1608Metric, F.Cu at (-3.28, -73.9)
- added C15: 100n, Capacitor_SMD:C_0603_1608Metric, F.Cu at (-3.28, -71.4)
- added C16: 10u, Capacitor_SMD:C_0603_1608Metric, F.Cu at (-3.28, -68.9)
- added C17: 10u, Capacitor_SMD:C_0603_1608Metric, F.Cu at (-3.28, -66.4)
- added C18: 22n, Capacitor_SMD:C_0603_1608Metric, F.Cu at (-3.28, -63.9)
- added C19: 100n, Capacitor_SMD:C_0603_1608Metric, F.Cu at (-3.28, -61.4)
- added C2: 100n, Capacitor_SMD:C_0603_1608Metric, F.Cu at (-7.29, -73.9)
- added C20: 100n, Capacitor_SMD:C_0603_1608Metric, F.Cu at (-3.28, -58.9)
- added C21: 10u, Capacitor_SMD:C_0603_1608Metric, F.Cu at (-3.28, -56.4)
- added C22: 10u, Capacitor_SMD:C_0603_1608Metric, F.Cu at (-3.28, -53.8)
- added C23: 10u, Capacitor_SMD:C_0603_1608Metric, F.Cu at (-3.28, -51.3)
- added C24: 10u, Capacitor_SMD:C_0603_1608Metric, F.Cu at (0.73, -76.4)
- added C25: 2u2, Capacitor_SMD:C_0603_1608Metric, F.Cu at (0.73, -73.9)
- added C26: 100n, Capacitor_SMD:C_0603_1608Metric, F.Cu at (0.73, -71.4)
- added C27: 10u, Capacitor_SMD:C_0603_1608Metric, F.Cu at (0.73, -68.9)
- added C28: 1u, Capacitor_SMD:C_0603_1608Metric, F.Cu at (80.3, -76.4)
- added C29: 100n, Capacitor_SMD:C_0603_1608Metric, F.Cu at (105.4, 59.2)
- added C3: 10u, Capacitor_SMD:C_0603_1608Metric, F.Cu at (-7.29, -71.4)
- added C30: 1u, Capacitor_SMD:C_0603_1608Metric, F.Cu at (80.3, -71.4)
- added C31: 100n, Capacitor_SMD:C_0603_1608Metric, F.Cu at (80.3, -68.9)
- added C32: 100n, Capacitor_SMD:C_0603_1608Metric, F.Cu at (1.96, -34.3)
- added C33: 2u2, Capacitor_SMD:C_0603_1608Metric, F.Cu at (1.96, -31.8)
- added C34: 2u2, Capacitor_SMD:C_0603_1608Metric, F.Cu at (1.96, -29.3)
- added C35: 10u, Capacitor_SMD:C_0603_1608Metric, F.Cu at (1.96, -26.8)
- added C36: 100n, Capacitor_SMD:C_0603_1608Metric, F.Cu at (1.96, -24.3)
- added C37: 100n, Capacitor_SMD:C_0603_1608Metric, F.Cu at (1.96, -21.8)
- added C38: 2u2, Capacitor_SMD:C_0603_1608Metric, F.Cu at (1.96, -19.3)
- added C39: 10u, Capacitor_SMD:C_0603_1608Metric, F.Cu at (1.96, -16.8)
- added C4: 10u, Capacitor_SMD:C_0603_1608Metric, F.Cu at (-7.29, -68.9)
- added C40: 2u2, Capacitor_SMD:C_0603_1608Metric, F.Cu at (1.96, -14.2)
- added C41: 100n, Capacitor_SMD:C_0603_1608Metric, F.Cu at (5.97, -34.3)
- added C42: 100n, Capacitor_SMD:C_0603_1608Metric, F.Cu at (5.97, -31.8)
- added C43: 10u, Capacitor_SMD:C_0603_1608Metric, F.Cu at (5.97, -29.3)
- added C44: 100u, Capacitor_THT:CP_Radial_D6.3mm_P2.50mm, F.Cu at (103.8, 79.0)
- added C45: 100n, Capacitor_SMD:C_0603_1608Metric, F.Cu at (5.97, -26.8)
- added C46: 100n, Capacitor_SMD:C_0603_1608Metric, F.Cu at (5.97, -24.3)
- added C47: 10u, Capacitor_SMD:C_0603_1608Metric, F.Cu at (5.97, -21.8)
- added C48: 100n, Capacitor_SMD:C_0603_1608Metric, F.Cu at (5.97, -19.3)
- added C49: 100n, Capacitor_SMD:C_0603_1608Metric, F.Cu at (5.97, -16.8)
- added C5: 220u, Capacitor_THT:CP_Radial_D6.3mm_P2.50mm, F.Cu at (158.2, 56.8)
- added C50: 10u, Capacitor_SMD:C_0603_1608Metric, F.Cu at (5.97, -14.2)
- added C51: 10u, Capacitor_SMD:C_0603_1608Metric, F.Cu at (9.98, -34.3)
- added C52: 10u, Capacitor_SMD:C_0603_1608Metric, F.Cu at (9.98, -31.8)
- added C53: 10u, Capacitor_SMD:C_0603_1608Metric, F.Cu at (9.98, -29.3)
- added C54: 10u, Capacitor_SMD:C_0603_1608Metric, F.Cu at (9.98, -26.8)
- added C55: 10u, Capacitor_SMD:C_0603_1608Metric, F.Cu at (9.98, -24.3)
- added C56: 100n, Capacitor_SMD:C_0603_1608Metric, F.Cu at (9.98, -21.8)
- added C57: 100n, Capacitor_SMD:C_0603_1608Metric, F.Cu at (9.98, -19.3)
- added C58: 100n, Capacitor_SMD:C_0603_1608Metric, F.Cu at (9.98, -16.8)
- added C59: 100n, Capacitor_SMD:C_0603_1608Metric, F.Cu at (9.98, -14.2)
- added C6: 10u, Capacitor_SMD:C_0603_1608Metric, F.Cu at (163.2, 57.5)
- added C60: 100n, Capacitor_SMD:C_0603_1608Metric, F.Cu at (14.0, -34.3)
- added C61: 100n, Capacitor_SMD:C_0603_1608Metric, F.Cu at (14.0, -31.8)
- added C62: 100n, Capacitor_SMD:C_0603_1608Metric, F.Cu at (14.0, -29.3)
- added C63: 100n, Capacitor_SMD:C_0603_1608Metric, F.Cu at (14.0, -26.8)
- added C64: 10u, Capacitor_SMD:C_0603_1608Metric, F.Cu at (14.0, -24.3)
- added C65: 10u, Capacitor_SMD:C_0603_1608Metric, F.Cu at (14.0, -21.8)
- added C66: 22n, Capacitor_SMD:C_0603_1608Metric, F.Cu at (14.0, -19.3)
- added C67: 1000p, Capacitor_SMD:C_0603_1608Metric, F.Cu at (14.0, -16.8)
- added C68: 10u, Capacitor_SMD:C_0603_1608Metric, F.Cu at (38.9, -32.6)
- added C69: 4u7, Capacitor_SMD:C_0603_1608Metric, F.Cu at (38.9, -30.1)
- added C7: np/100n, Capacitor_SMD:C_0603_1608Metric, F.Cu at (-7.29, -63.9)
- added C70: 10u, Capacitor_SMD:C_0603_1608Metric, F.Cu at (38.9, -27.6)
- added C71: 100n, Capacitor_SMD:C_0603_1608Metric, F.Cu at (38.9, -25.0)
- added C72: 100n, Capacitor_SMD:C_0603_1608Metric, F.Cu at (38.9, -22.5)
- added C73: 10u, Capacitor_SMD:C_0603_1608Metric, F.Cu at (38.9, -20.0)
- added C74: 4u7, Capacitor_SMD:C_0603_1608Metric, F.Cu at (38.9, -17.5)
- added C75: 10u, Capacitor_SMD:C_0603_1608Metric, F.Cu at (42.9, -32.6)
- added C76: 4u7, Capacitor_SMD:C_0603_1608Metric, F.Cu at (42.9, -30.1)
- added C77: 10u, Capacitor_SMD:C_0603_1608Metric, F.Cu at (42.9, -27.6)
- added C78: 100n, Capacitor_SMD:C_0603_1608Metric, F.Cu at (59.7, -49.6)
- added C79: 10u, Capacitor_SMD:C_0603_1608Metric, F.Cu at (59.7, -47.1)
- added C8: 10u, Capacitor_SMD:C_0603_1608Metric, F.Cu at (-7.29, -61.4)
- added C80: 10u, Capacitor_SMD:C_0603_1608Metric, F.Cu at (59.7, -44.6)
- added C81: 100n, Capacitor_SMD:C_0603_1608Metric, F.Cu at (59.7, -42.1)
- added C82: 100n, Capacitor_SMD:C_0603_1608Metric, F.Cu at (59.7, -39.6)
- added C83: 100n, Capacitor_SMD:C_0603_1608Metric, F.Cu at (59.7, -37.1)
- added C84: 5100p, Capacitor_SMD:C_0603_1608Metric, F.Cu at (70.2, -24.5)
- added C85: 5100p, Capacitor_SMD:C_0603_1608Metric, F.Cu at (70.2, -22.0)
- added C86: 2700p, Capacitor_SMD:C_0603_1608Metric, F.Cu at (70.2, -19.4)
- added C87: 2700p, Capacitor_SMD:C_0603_1608Metric, F.Cu at (70.2, -16.9)
- added C88: 2700p, Capacitor_SMD:C_0603_1608Metric, F.Cu at (70.2, -14.4)
- added C89: 2700p, Capacitor_SMD:C_0603_1608Metric, F.Cu at (70.2, -11.9)
- added C9: 100n, Capacitor_SMD:C_0603_1608Metric, F.Cu at (-7.29, -58.9)
- added C90: 100n, Capacitor_SMD:C_0603_1608Metric, F.Cu at (70.2, -9.41)
- added C91: np/2n7, Capacitor_SMD:C_0603_1608Metric, F.Cu at (70.2, -6.90)
- added C92: 100n, Capacitor_SMD:C_0603_1608Metric, F.Cu at (70.2, -4.39)
- added C93: np/2n7, Capacitor_SMD:C_0603_1608Metric, F.Cu at (74.2, -24.5)
- added C94: 10u, Capacitor_SMD:C_0603_1608Metric, F.Cu at (74.2, -22.0)
- added C95: 10u, Capacitor_SMD:C_0603_1608Metric, F.Cu at (74.2, -19.4)
- added C96: 100n, Capacitor_SMD:C_0603_1608Metric, F.Cu at (74.2, -16.9)
- added C97: 100n, Capacitor_SMD:C_0603_1608Metric, F.Cu at (74.2, -14.4)
- added C98: 10u, Capacitor_SMD:C_0603_1608Metric, F.Cu at (74.2, -11.9)
- added C99: 10u, Capacitor_SMD:C_0603_1608Metric, F.Cu at (74.2, -9.41)
- added D1: LED_Small, LED_SMD:LED_0603_1608Metric, F.Cu at (31.6, -39.9)
- added D2: LED_Small, LED_SMD:LED_0603_1608Metric, F.Cu at (70.3, -57.0)
- added J1: DCJ200-05-A, LNIC_Connector_BarrelJack:DCJ200-05-A, F.Cu at (147.2, 58.4)
- added J10: Conn_01x03, Connector_PinHeader_2.54mm:PinHeader_1x03_P2.54mm_Vertical, F.Cu at (56.1, -15.3)
- added J2: Conn_01x02, Connector_PinHeader_2.54mm:PinHeader_1x02_P2.54mm_Vertical, F.Cu at (31.9, -46.0)
- added J4: Conn_02x03_Counter_Clockwise, Connector_PinHeader_2.54mm:PinHeader_2x03_P2.54mm_Vertical, F.Cu at (70.6, -65.7)
- added J5: Conn_01x03, Connector_PinHeader_2.54mm:PinHeader_1x03_P2.54mm_Vertical, F.Cu at (60.0, -75.4)
- added J6: Conn_01x03, Connector_PinHeader_2.54mm:PinHeader_1x03_P2.54mm_Vertical, F.Cu at (64.7, -75.4)
- added J7: Conn_01x03, Connector_PinHeader_2.54mm:PinHeader_1x03_P2.54mm_Vertical, F.Cu at (69.3, -75.4)
- added J8: Conn_01x03, Connector_PinHeader_2.54mm:PinHeader_1x03_P2.54mm_Vertical, F.Cu at (74.0, -75.4)
- added J9: Conn_01x10, Connector_PinHeader_2.54mm:PinHeader_1x10_P2.54mm_Vertical, F.Cu at (28.4, -33.3)
- added L2: 104CDMCCDS-330MC, LNIC_Inductor_SMD:L_Sumida_104CDMCCDS, F.Cu at (171.9, 55.8)
- added L3: L_Eaton_HCM1A0805-470-R, LNIC_Inductor_SMD:L_Eaton_HCM1A0805, F.Cu at (188.2, 69.4)
- added L4: ASPI-6045T-220M-T, LNIC_Inductor_SMD:L_Abracon_ASPI-6045T, F.Cu at (59.0, -58.2)
- added L5: ASPI-6045T-220M-T, LNIC_Inductor_SMD:L_Abracon_ASPI-6045T, F.Cu at (-4.67, -31.5)
- added L6: ASPI-6045T-220M-T, LNIC_Inductor_SMD:L_Abracon_ASPI-6045T, F.Cu at (-4.67, -23.4)
- added L7: ASPI-6045T-220M-T, LNIC_Inductor_SMD:L_Abracon_ASPI-6045T, F.Cu at (-4.67, -15.3)
- added L8: ASPI-6045T-220M-T, LNIC_Inductor_SMD:L_Abracon_ASPI-6045T, F.Cu at (92.2, 118.9)
- added L9: ASPI-6045T-220M-T, LNIC_Inductor_SMD:L_Abracon_ASPI-6045T, F.Cu at (129.7, 86.6)
- added Q1: BSN20, Package_TO_SOT_SMD:SOT-23, F.Cu at (51.3, -15.4)
- added Q2: BSN20, Package_TO_SOT_SMD:SOT-23, F.Cu at (51.3, -10.9)
- added Q3: BSN20, Package_TO_SOT_SMD:SOT-23, F.Cu at (51.3, -6.46)
- added R1: 4k7, Resistor_SMD:R_0603_1608Metric, F.Cu at (80.3, -58.2)
- added R10: 10k, Resistor_SMD:R_0603_1608Metric, F.Cu at (4.74, -76.4)
- added R11: 91k, Resistor_SMD:R_0603_1608Metric, F.Cu at (4.74, -73.9)
- added R12: 0R, Resistor_SMD:R_0603_1608Metric, F.Cu at (4.74, -71.4)
- added R13: 680R, Resistor_SMD:R_0603_1608Metric, F.Cu at (4.74, -68.9)
- added R14: 33k, Resistor_SMD:R_0603_1608Metric, F.Cu at (4.74, -66.4)
- added R15: 10k, Resistor_SMD:R_0603_1608Metric, F.Cu at (4.74, -63.9)
- added R16: 0R, Resistor_SMD:R_0603_1608Metric, F.Cu at (4.74, -61.4)
- added R17: 0R, Resistor_SMD:R_0603_1608Metric, F.Cu at (4.74, -58.9)
- added R18: 0R, Resistor_SMD:R_0603_1608Metric, F.Cu at (4.74, -56.4)
- added R19: 91k, Resistor_SMD:R_0603_1608Metric, F.Cu at (4.74, -53.8)
- added R2: 4k7, Resistor_SMD:R_0603_1608Metric, F.Cu at (80.3, -55.7)
- added R20: 15k, Resistor_SMD:R_0603_1608Metric, F.Cu at (4.74, -51.3)
- added R21: 10k, Resistor_SMD:R_0603_1608Metric, F.Cu at (8.75, -76.4)
- added R22: 10k, Resistor_SMD:R_0603_1608Metric, F.Cu at (8.75, -73.9)
- added R23: 10k, Resistor_SMD:R_0603_1608Metric, F.Cu at (8.75, -71.4)
- added R24: 330R, Resistor_SMD:R_0603_1608Metric, F.Cu at (8.75, -68.9)
- added R25: 18k, Resistor_SMD:R_0603_1608Metric, F.Cu at (8.75, -66.4)
- added R26: 10k, Resistor_SMD:R_0603_1608Metric, F.Cu at (8.75, -63.9)
- added R27: np/0R, Resistor_SMD:R_0603_1608Metric, F.Cu at (80.3, -66.4)
- added R28: 0R, Resistor_SMD:R_0603_1608Metric, F.Cu at (80.3, -63.9)
- added R29: R_Small, Resistor_SMD:R_0603_1608Metric, F.Cu at (14.0, -14.2)
- added R3: 10k, Resistor_SMD:R_0603_1608Metric, F.Cu at (0.73, -66.4)
- added R30: 0R, Resistor_SMD:R_0603_1608Metric, F.Cu at (18.0, -34.3)
- added R31: 0R, Resistor_SMD:R_0603_1608Metric, F.Cu at (18.0, -31.8)
- added R32: 0R, Resistor_SMD:R_0603_1608Metric, F.Cu at (18.0, -29.3)
- added R33: 0R, Resistor_SMD:R_0603_1608Metric, F.Cu at (18.0, -26.8)
- added R34: 0R, Resistor_SMD:R_0603_1608Metric, F.Cu at (18.0, -24.3)
- added R35: 1k37, Resistor_SMD:R_0603_1608Metric, F.Cu at (18.0, -21.8)
- added R36: 0R, Resistor_SMD:R_0603_1608Metric, F.Cu at (18.0, -19.3)
- added R37: 10k, Resistor_SMD:R_0603_1608Metric, F.Cu at (18.0, -16.8)
- added R38: 10k, Resistor_SMD:R_0603_1608Metric, F.Cu at (42.9, -25.0)
- added R39: np/0R, Resistor_SMD:R_0603_1608Metric, F.Cu at (42.9, -22.5)
- added R4: 33k, Resistor_SMD:R_0603_1608Metric, F.Cu at (0.73, -63.9)
- added R40: np/0R, Resistor_SMD:R_0603_1608Metric, F.Cu at (42.9, -20.0)
- added R41: 10k, Resistor_SMD:R_0603_1608Metric, F.Cu at (42.9, -17.5)
- added R42: 0R, Resistor_SMD:R_0603_1608Metric, F.Cu at (46.9, -32.6)
- added R43: 10k, Resistor_SMD:R_0603_1608Metric, F.Cu at (46.9, -30.1)
- added R44: 10k, Resistor_SMD:R_0603_1608Metric, F.Cu at (46.9, -27.6)
- added R45: 0R, Resistor_SMD:R_0603_1608Metric, F.Cu at (46.9, -25.0)
- added R46: 0R, Resistor_SMD:R_0603_1608Metric, F.Cu at (46.9, -22.5)
- added R47: 10k, Resistor_SMD:R_0603_1608Metric, F.Cu at (63.7, -49.6)
- added R48: 330R, Resistor_SMD:R_0603_1608Metric, F.Cu at (63.7, -47.1)
- added R49: 0R, Resistor_SMD:R_0603_1608Metric, F.Cu at (63.7, -44.6)
- added R5: 10k, Resistor_SMD:R_0603_1608Metric, F.Cu at (0.73, -61.4)
- added R50: 0R, Resistor_SMD:R_0603_1608Metric, F.Cu at (63.7, -42.1)
- added R51: 0R, Resistor_SMD:R_0603_1608Metric, F.Cu at (63.7, -39.6)
- added R52: np/100k, Resistor_SMD:R_0603_1608Metric, F.Cu at (63.7, -37.1)
- added R53: np/100k, Resistor_SMD:R_0603_1608Metric, F.Cu at (67.7, -49.6)
- added R54: np/100k, Resistor_SMD:R_0603_1608Metric, F.Cu at (67.7, -47.1)
- added R55: np/100k, Resistor_SMD:R_0603_1608Metric, F.Cu at (67.7, -44.6)
- added R56: 10k, Resistor_SMD:R_0603_1608Metric, F.Cu at (67.7, -42.1)
- added R57: 10k, Resistor_SMD:R_0603_1608Metric, F.Cu at (67.7, -39.6)
- added R58: 1k, Resistor_SMD:R_0603_1608Metric, F.Cu at (74.2, -6.90)
- added R59: 1k, Resistor_SMD:R_0603_1608Metric, F.Cu at (74.2, -4.39)
- added R6: np/0R, Resistor_SMD:R_0603_1608Metric, F.Cu at (0.73, -58.9)
- added R60: 1k, Resistor_SMD:R_0603_1608Metric, F.Cu at (78.3, -24.5)
- added R61: 1k, Resistor_SMD:R_0603_1608Metric, F.Cu at (78.3, -22.0)
- added R62: 1k1, Resistor_SMD:R_0603_1608Metric, F.Cu at (78.3, -19.4)
- added R63: 1k1, Resistor_SMD:R_0603_1608Metric, F.Cu at (78.3, -16.9)
- added R64: 1k1, Resistor_SMD:R_0603_1608Metric, F.Cu at (78.3, -14.4)
- added R65: 1k1, Resistor_SMD:R_0603_1608Metric, F.Cu at (78.3, -11.9)
- added R66: 1k1, Resistor_SMD:R_0603_1608Metric, F.Cu at (78.3, -9.41)
- added R67: 1k1, Resistor_SMD:R_0603_1608Metric, F.Cu at (78.3, -6.90)
- added R68: 1k1, Resistor_SMD:R_0603_1608Metric, F.Cu at (78.3, -4.39)
- added R69: 1k1, Resistor_SMD:R_0603_1608Metric, F.Cu at (82.3, -24.5)
- added R7: 0R, Resistor_SMD:R_0603_1608Metric, F.Cu at (0.73, -56.4)
- added R70: 0R, Resistor_SMD:R_0603_1608Metric, F.Cu at (82.3, -22.0)
- added R71: 0R, Resistor_SMD:R_0603_1608Metric, F.Cu at (82.3, -19.4)
- added R72: 0R, Resistor_SMD:R_0603_1608Metric, F.Cu at (82.3, -16.9)
- added R73: 0R, Resistor_SMD:R_0603_1608Metric, F.Cu at (82.3, -14.4)
- added R74: 10k, Resistor_SMD:R_0603_1608Metric, F.Cu at (82.3, -11.9)
- added R75: 10k, Resistor_SMD:R_0603_1608Metric, F.Cu at (82.3, -9.41)
- added R76: 10k, Resistor_SMD:R_0603_1608Metric, F.Cu at (32.7, -34.3)
- added R8: np/0R, Resistor_SMD:R_0603_1608Metric, F.Cu at (0.73, -53.8)
- added R9: 10k, Resistor_SMD:R_0603_1608Metric, F.Cu at (0.73, -51.3)
- added SW1: SW_SPST, Button_Switch_THT:SW_PUSH_6mm, F.Cu at (177.1, 121.2)
- added SW2: SW_SPST, Button_Switch_THT:SW_PUSH_6mm, F.Cu at (195.9, 125.8)
- added TP1: TestPoint, TestPoint:TestPoint_Pad_D2.0mm, F.Cu at (-7.27, -48.0)
- added TP10: TestPoint, TestPoint:TestPoint_Pad_D2.0mm, F.Cu at (64.2, -31.8)
- added TP11: TestPoint, TestPoint:TestPoint_Pad_D2.0mm, F.Cu at (64.2, -27.8)
- added TP12: TestPoint, TestPoint:TestPoint_Pad_D2.0mm, F.Cu at (64.2, -23.7)
- added TP13: TestPoint, TestPoint:TestPoint_Pad_D2.0mm, F.Cu at (70.3, -31.8)
- added TP14: TestPoint, TestPoint:TestPoint_Pad_D2.0mm, F.Cu at (70.3, -27.8)
- added TP15: TestPoint, TestPoint:TestPoint_Pad_D2.0mm, F.Cu at (74.3, -31.8)
- added TP16: TestPoint, TestPoint:TestPoint_Pad_D2.0mm, F.Cu at (74.3, -27.8)
- added TP17: TestPoint, TestPoint:TestPoint_Pad_D2.0mm, F.Cu at (78.4, -31.8)
- added TP18: TestPoint, TestPoint:TestPoint_Pad_D2.0mm, F.Cu at (78.4, -27.8)
- added TP19: TestPoint, TestPoint:TestPoint_Pad_D2.0mm, F.Cu at (82.4, -31.8)
- added TP2: TestPoint, TestPoint:TestPoint_Pad_D2.0mm, F.Cu at (-7.27, -44.0)
- added TP20: TestPoint, TestPoint:TestPoint_Pad_D2.0mm, F.Cu at (82.4, -27.8)
- added TP21: TestPoint, TestPoint:TestPoint_Pad_D2.0mm, F.Cu at (22.0, -29.5)
- added TP22: TestPoint, TestPoint:TestPoint_Pad_D2.0mm, F.Cu at (22.0, -25.5)
- added TP23: TestPoint, TestPoint:TestPoint_Pad_D2.0mm, F.Cu at (22.0, -21.4)
- added TP24: TestPoint, TestPoint:TestPoint_Pad_D2.0mm, F.Cu at (22.0, -17.4)
- added TP25: TestPoint, TestPoint:TestPoint_Pad_D2.0mm, F.Cu at (-3.22, -44.0)
- added TP26: TestPoint, TestPoint:TestPoint_Pad_D2.0mm, F.Cu at (-3.22, -40.0)
- added TP27: TestPoint, TestPoint:TestPoint_Pad_D2.0mm, F.Cu at (0.83, -48.0)
- added TP28: TestPoint, TestPoint:TestPoint_Pad_D2.0mm, F.Cu at (0.83, -44.0)
- added TP29: TestPoint, TestPoint:TestPoint_Pad_D2.0mm, F.Cu at (0.83, -40.0)
- added TP3: TestPoint, TestPoint:TestPoint_Pad_D2.0mm, F.Cu at (-7.27, -40.0)
- added TP30: TestPoint, TestPoint:TestPoint_Pad_D2.0mm, F.Cu at (4.88, -48.0)
- added TP31: TestPoint, TestPoint:TestPoint_Pad_D2.0mm, F.Cu at (4.88, -44.0)
- added TP32: TestPoint, TestPoint:TestPoint_Pad_D2.0mm, F.Cu at (4.88, -40.0)
- added TP33: TestPoint, TestPoint:TestPoint_Pad_D2.0mm, F.Cu at (84.3, -67.5)
- added TP34: TestPoint, TestPoint:TestPoint_Pad_D2.0mm, F.Cu at (84.3, -63.5)
- added TP4: TestPoint, TestPoint:TestPoint_Pad_D2.0mm, F.Cu at (-3.22, -48.0)
- added TP5: TestPoint, TestPoint:TestPoint_Pad_D2.0mm, F.Cu at (22.0, -33.6)
- added TP6: TestPoint, TestPoint:TestPoint_Pad_D2.0mm, F.Cu at (60.2, -31.8)
- added TP7: TestPoint, TestPoint:TestPoint_Pad_D2.0mm, F.Cu at (60.2, -27.8)
- added TP8: TestPoint, TestPoint:TestPoint_Pad_D2.0mm, F.Cu at (60.2, -23.7)
- added TP9: TestPoint, TestPoint:TestPoint_Pad_D2.0mm, F.Cu at (60.2, -19.6)
- added U1: LDL212DR, Package_SO:SO-8_3.9x4.9mm_P1.27mm, F.Cu at (128.8, 74.0)
- added U10: TSDP11XX, Package_DFN_QFN:QFN-20-1EP_4x4mm_P0.5mm_EP2.5x2.5mm, F.Cu at (114.3, 110.8)
- added U11: ESP32-WROVER, LNIC_MCU:ESP32_WROVER_no_thermal_via, F.Cu at (183.9, 106.5)
- added U12: OPA1632DGN, LNIC_Package_SO:VSSOP-8_3.0x3.0mm_P0.65mm_EP1.57x1.89mm, F.Cu at (109.9, 97.6)
- added U13: OPA1632DGN, LNIC_Package_SO:VSSOP-8_3.0x3.0mm_P0.65mm_EP1.57x1.89mm, F.Cu at (118.5, 97.6)
- added U3: RT7272A, Package_SO:SOIC-8-1EP_3.9x4.9mm_P1.27mm_EP2.41x3.3mm_ThermalVias, F.Cu at (191.2, 60.2)
- added U4: LDL212DR, Package_SO:SO-8_3.9x4.9mm_P1.27mm, F.Cu at (129.4, 96.2)
- added U6: LDL212DR, Package_SO:SO-8_3.9x4.9mm_P1.27mm, F.Cu at (156.5, 83.2)
- added U8: 74AHCT1G126, Package_TO_SOT_SMD:SOT-353_SC-70-5_Handsoldering, F.Cu at (105.2, 63.6)
- added X1: ECS-2520MV-xxx-xx, Oscillator:Oscillator_SMD_ECS_2520MV-xxx-xx-4Pin_2.5x2.0mm, F.Cu at (11.6, -10.8)
- added np/R1: 18k, Resistor_SMD:R_0603_1608Metric, F.Cu at (8.75, -61.4)
- added np/R2: 56k, Resistor_SMD:R_0603_1608Metric, F.Cu at (8.75, -58.9)
- U5: value MAX13331 -> LP2951-5.0_SOIC; footprint Package_SO:QSOP-16_3.9x4.9mm_P0.635mm -> Package_SO:SOIC-8_3.9x4.9mm_P1.27mm
- moved R1 80.3 mm to (98.2, -8.75)
- moved R10 80.3 mm to (100.7, -8.75)
- moved R11 80.3 mm to (100.7, -7.00)
- moved R12 80.3 mm to (100.7, -5.25)
- moved R13 80.3 mm to (100.7, -3.50)
- moved R14 80.3 mm to (100.7, -1.75)
- moved R15 80.3 mm to (100.7, 0.00)
- moved R16 80.3 mm to (100.7, 1.75)
- moved R17 80.3 mm to (103.1, -8.75)
- moved R18 80.3 mm to (103.1, -7.00)
- moved R19 80.3 mm to (103.1, -5.25)
- moved R2 80.3 mm to (98.2, -7.00)
- moved R20 80.3 mm to (103.1, -3.50)
- moved R3 80.3 mm to (98.2, -5.25)
- moved R6 80.3 mm to (98.2, -3.50)
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- renumbered U3 to U2, U11 to U9
Connections:
- U2 pad 1: unconnected-(U3-FC-Pad1) -> Net-(U2-FC)
- U2 pad 2: unconnected-(U3-CAP+-Pad2) -> Net-(U2-CAP+)
- U2 pad 4: unconnected-(U3-CAP--Pad4) -> Net-(U2-CAP-)
- U2 pad 6: unconnected-(U3-LV-Pad6) -> Net-(U2-LV)
- U2 pad 7: unconnected-(U3-OSC-Pad7) -> Net-(U2-OSC)
- U2 pad 8: +5V5 -> Net-(U2-V+)
- U5 pad 1: unconnected-(U5-INL-Pad1) -> Net-(U5-OUT)
- U5 pad 2: unconnected-(U5-SGND-Pad2) -> Net-(U5-SENSE)
- U5 pad 3: unconnected-(U5-INR-Pad3) -> Net-(U5-SHUTDOWN)
- U5 pad 4: unconnected-(U5-SGND-Pad4) -> Net-(U5-GND)
- U5 pad 5: unconnected-(U5-VDD-Pad5) -> Net-(U5-~{ERROR})
- U5 pad 6: unconnected-(U5-~{SHDN}-Pad6) -> Net-(U5-VTAP)
- U5 pad 7: unconnected-(U5-CPVDD-Pad7) -> Net-(U5-FEEDBACK)
- U5 pad 8: unconnected-(U5-C1P-Pad8) -> +5V5
- U7 pad 1: unconnected-(U7-OUT-Pad1) -> Net-(U7-OUT)
- U7 pad 2: unconnected-(U7-GND-Pad2) -> GND
- U7 pad 3: unconnected-(U7-VCC-Pad3) -> Net-(U7-VCC)
- U9 pad 1: unconnected-(U11-CX_SDIN1-Pad1) -> /Codec/CX_SDIN1
- U9 pad 11: /Codec/CS42528_INT -> /Codec/CODEC_INT
- U9 pad 12: /Codec/CS42528_nRST -> /Codec/~{RST}
- U9 pad 13: /Codec/AINR- -> unconnected-(U9-AINR--Pad13)
- U9 pad 14: /Codec/AINR+ -> unconnected-(U9-AINR+-Pad14)
- U9 pad 15: /Codec/AINL+ -> unconnected-(U9-AINL+-Pad15)
- U9 pad 16: /Codec/AINL- -> unconnected-(U9-AINL--Pad16)
- U9 pad 18: unconnected-(U11-FILT+-Pad18) -> /Codec/FILT+
- U9 pad 19: unconnected-(U11-REFGND-Pad19) -> GND
- U9 pad 2: unconnected-(U11-CX_SCLK-Pad2) -> /Codec/CX_SCLK
- U9 pad 3: unconnected-(U11-CX_LRCK-Pad3) -> /Codec/CX_LRCK
- U9 pad 30: /Codec/AOUTB2- -> unconnected-(U9-AOUTB2--Pad30)
- U9 pad 31: /Codec/AOUTB2+ -> unconnected-(U9-AOUTB2+-Pad31)
- U9 pad 34: unconnected-(U11-AOUTB1--Pad34) -> /Codec/AOUTB1-
- U9 pad 35: unconnected-(U11-AOUTB1+-Pad35) -> /Codec/AOUTB1+
- U9 pad 38: Net-(U11-MUTEC) -> /Codec/MUTEC_0
- U9 pad 39: unconnected-(U11-LPFLT-Pad39) -> /Codec/LPFLT
- U9 pad 41: +5VA -> Net-(U9-VARX)
- U9 pad 42: GND -> Net-(U9-RXP7/GPO7)
- U9 pad 43: GND -> Net-(U9-RXP6/GPO6)
- U9 pad 44: GND -> Net-(U9-RXP5/GPO5)
- U9 pad 45: GND -> Net-(U9-RXP4/GPO4)
- U9 pad 46: unconnected-(U11-RXP3/GPO3-Pad46) -> Net-(U9-RXP3/GPO3)
- U9 pad 47: unconnected-(U11-RXP2/GPO2-Pad47) -> Net-(U9-RXP2/GPO2)
- U9 pad 48: unconnected-(U11-RXP1/GPO1-Pad48) -> Net-(U9-RXP1/GPO1)
- U9 pad 49: /Codec/SPDIF_RXP0 -> /Input/SPDIF_DATA
- U9 pad 59: unconnected-(U11-OMCK-Pad59) -> /Codec/OSC_OMCK
Other:
- board size 54 x 80 mm -> 100 x 80 mm
- copper layers 2 -> 4
- board text added: "1.4mm from edge of pcb to front / back plate + 1.6mm thickness of back plate"
- board text added: "1.4mm gap"
- board text added: "1.6mm front panel"

Commit message: layout init
Parts:
- removed J9: Conn_01x10, Connector_PinHeader_2.54mm:PinHeader_1x10_P2.54mm_Vertical
- removed L5, L6, L7, L8, L9: ASPI-6045T-220M-T, LNIC_Inductor_SMD:L_Abracon_ASPI-6045T
- removed the R1 at (98.2, -8.75)
- removed the R10 at (100.7, -8.75)
- removed the R11 at (100.7, -7.00)
- removed the R12 at (100.7, -5.25)
- removed the R13 at (100.7, -3.50)
- removed the R14 at (100.7, -1.75)
- removed the R15 at (100.7, 0.00)
- removed the R16 at (100.7, 1.75)
- removed the R17 at (103.1, -8.75)
- removed the R18 at (103.1, -7.00)
- removed the R19 at (103.1, -5.25)
- removed the R2 at (98.2, -7.00)
- removed the R20 at (103.1, -3.50)
- removed the R3 at (98.2, -5.25)
- removed the R36 at (18.0, -19.3)
- removed the R37 at (18.0, -16.8)
- removed R45, R46: 0R, Resistor_SMD:R_0603_1608Metric
- removed R52, R53, R54, R55: np/100k, Resistor_SMD:R_0603_1608Metric
- removed the R6 at (98.2, -3.50)
- removed the R7 at (98.2, -1.75)
- removed the R8 at (98.2, 0.00)
- removed the R9 at (98.2, 1.75)
- removed SW1, SW2: SW_SPST, Button_Switch_THT:SW_PUSH_6mm
- removed TP1, TP10, TP11, TP12, TP13, TP14, TP15, TP16, TP17, TP18, TP19, TP2, TP20, TP21, TP22, TP23, TP24, TP25, TP26, TP27, TP28, TP29, TP3, TP30, TP31, TP32, TP33, TP34, TP4, TP5, TP6, TP7, TP8, TP9: TestPoint, TestPoint:TestPoint_Pad_D2.0mm
- added C100: np/10u, Capacitor_SMD:C_0603_1608Metric, F.Cu at (185.5, 59.7)
- added C101: np/10u, Capacitor_SMD:C_0603_1608Metric, F.Cu at (173.6, 66.7)
- added C102: 10u, Capacitor_SMD:C_0603_1608Metric, F.Cu at (134.0, 121.5)
- added C103: 10u, Capacitor_SMD:C_0603_1608Metric, F.Cu at (131.4, 118.4)
- added C104: 10u, Capacitor_SMD:C_0603_1608Metric, F.Cu at (158.8, 89.7)
- added C105: np/10u, Capacitor_SMD:C_0603_1608Metric, F.Cu at (148.1, 82.2)
- added C106: np/10u, Capacitor_SMD:C_0603_1608Metric, F.Cu at (148.1, 72.9)
- added C107: np/10u, Capacitor_SMD:C_0603_1608Metric, F.Cu at (158.8, 70.8)
- added C108: np/10u, Capacitor_SMD:C_0603_1608Metric, F.Cu at (158.8, 80.2)
- added H1: MountingHole, MountingHole:MountingHole_3.2mm_M3, F.Cu at (51.7, 35.3)
- added H2: MountingHole, MountingHole:MountingHole_3.2mm_M3, F.Cu at (45.7, 40.7)
- added H3: MountingHole, MountingHole:MountingHole_3.2mm_M3, F.Cu at (44.9, 32.8)
- added H4: MountingHole, MountingHole:MountingHole_3.2mm_M3, F.Cu at (105.7, 53.5)
- added J11: NRJ6HM-1-PRE, LNIC_Connector_Audio:Jack_6.35mm_Neutrik_NRJ6HM-1-PRE_Horizontal, F.Cu at (117.9, 113.7)
- added J3: Conn_02x03_Odd_Even, Connector_PinHeader_2.54mm:PinHeader_2x03_P2.54mm_Vertical, F.Cu at (172.7, 95.4)
- added RV1: R_Potentiometer, LNIC_Potentiometer_THT:Potentiometer_Bourns_PTD901-XX15K-X_Horizontal, F.Cu at (161.8, 131.1)
- C33: value 2u2 -> np/10u
- C34: value 2u2 -> 10u
- R31: value 0R -> np/0R
- R36: renamed from np/R1; value 18k -> np/18k
- R37: renamed from np/R2; value 56k -> np/56k
- U3: footprint Package_SO:SOIC-8-1EP_3.9x4.9mm_P1.27mm_EP2.41x3.3mm_ThermalVias -> Package_SO:SOIC-8-1EP_3.9x4.9mm_P1.27mm_EP2.41x3.3mm
- moved C13 249.8 mm to (159.9, 112.7), turned to -90 degrees
- moved C4 247.9 mm to (161.5, 112.7), turned to -90 degrees
- moved C7 242.7 mm to (156.9, 114.8), turned to -90 degrees
- moved C14 242.0 mm to (150.9, 112.7), turned to -90 degrees
- moved C9 237.6 mm to (191.8, 70.8)
- moved C17 237.3 mm to (152.5, 112.7), turned to -90 degrees
- moved R6 236.2 mm to (163.1, 112.7), turned to -90 degrees
- moved C19 233.1 mm to (188.7, 70.8)
- moved R12 233.0 mm to (159.1, 103.1), turned to 180 degrees
- moved C25 232.8 mm to (160.4, 95.5), turned to 180 degrees
- moved R7 232.2 mm to (163.1, 109.7), turned to 90 degrees
- moved C16 230.2 mm to (185.5, 62.9), turned to 180 degrees
- moved R22 230.2 mm to (166.3, 93.9), turned to 90 degrees
- moved C20 229.7 mm to (193.5, 59.7)
- moved C10 229.1 mm to (155.5, 104.8), turned to 180 degrees
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Connections:
- net Net-(U3-SW) renamed /Supply/DCDC_SW
- net Net-(U7-VCC) renamed /Input/OPT_VCC
- C12 pad 1: Net-(U3-VIN) -> /Supply/DCDC_IN
- C16 pad 1: Net-(U3-VIN) -> /Supply/DCDC_IN
- C33 pad 1: +5V -> +5VA
- C34 pad 1: Net-(C34-Pad1) -> +5V
- C35 pad 1: Net-(C34-Pad1) -> +5V
- C36 pad 1: Net-(C34-Pad1) -> +5V
- C49 pad 1: Net-(C49-Pad1) -> +5V
- C52 pad 1: Net-(C49-Pad1) -> +5V
- C55 pad 1: Net-(U9-VARX) -> +5VA
- C56 pad 1: Net-(U9-VARX) -> +5VA
- C64 pad 1: Net-(U9-VARX) -> +5VA
- C70 pad 1: Net-(C70-Pad1) -> /Supply/DCDC_IN
- C71 pad 1: Net-(C70-Pad1) -> +5VA
- C72 pad 1: Net-(C72-Pad1) -> +5VA
- C73 pad 1: Net-(C72-Pad1) -> +5VA
- C74 pad 2: GND -> GND2
- C76 pad 2: GND -> GND2
- C77 pad 2: GND -> GND2
- C8 pad 1: Net-(U3-VIN) -> /Supply/DCDC_IN
- C91 pad 1: /Amplifier/FILT_RIGHT_N -> /Amplifier/FILT_RIGHT_P
- C91 pad 2: /Amplifier/FILT_RIGHT_P -> /Amplifier/FILT_RIGHT_N
- C93 pad 1: /Amplifier/FILT_LEFT_N -> /Amplifier/FILT_LEFT_P
- C93 pad 2: /Amplifier/FILT_LEFT_P -> /Amplifier/FILT_LEFT_N
- J10 pad 1: Net-(J10-Pin_1) -> /Amplifier/HP_L_0
- J10 pad 2: Net-(J10-Pin_2) -> /Amplifier/HP_R_0
- J10 pad 3: unconnected-(J10-Pin_3-Pad3) -> GND2
- L2 pad 2: Net-(U3-VIN) -> /Supply/DCDC_IN
- Q2 pad 2: /Amplifier/SDA -> /Amplifier/SDA_1
- Q3 pad 2: /Amplifier/SCL -> /Amplifier/SCL_1
- R1 pad 2: /Codec/SDA_1 -> /Amplifier/SDA_1
- R2 pad 2: /Codec/SCL_1 -> /Amplifier/SCL_1
- R39 pad 1: /Amplifier/SDA -> /Amplifier/SDA_1
- R40 pad 1: /Amplifier/SCL -> /Amplifier/SCL_1
- R58 pad 1: /Codec/AOUTA1- -> /Codec/AOUTA+
- R59 pad 1: /Codec/AOUTA1+ -> /Codec/AOUTA-
- R60 pad 1: /Codec/AOUTB1- -> /Codec/AOUTB+
- R61 pad 1: /Codec/AOUTB1+ -> /Codec/AOUTB-
- R70 pad 2: /Amplifier/FILT_RIGHT_N -> /Amplifier/FILT_RIGHT_P
- R71 pad 2: /Amplifier/FILT_RIGHT_P -> /Amplifier/FILT_RIGHT_N
- R72 pad 2: /Amplifier/FILT_LEFT_N -> /Amplifier/FILT_LEFT_P
- R73 pad 2: /Amplifier/FILT_LEFT_P -> /Amplifier/FILT_LEFT_N
- R9 pad 1: Net-(U3-VIN) -> /Supply/DCDC_IN
- U10 pad 11: Net-(U10-CP_GND) -> GND2
- U10 pad 15: Net-(C70-Pad1) -> +5VA
- U10 pad 18: Net-(C72-Pad1) -> +5VA
- U10 pad 7: Net-(U10-HP_L) -> /Amplifier/HP_L_0
- U10 pad 8: Net-(U10-HP_R) -> /Amplifier/HP_R_0
- U11 pad 12: /Control/TOUCH_2 -> unconnected-(U11-IO27-Pad12)
- U11 pad 13: /Control/TOUCH_3 -> unconnected-(U11-IO14-Pad13)
- U11 pad 16: /Control/TOUCH_4 -> unconnected-(U11-IO13-Pad16)
- U11 pad 33: /Codec/SDA_1 -> /Amplifier/SDA_1
- U11 pad 36: /Codec/SCL_1 -> /Amplifier/SCL_1
- U3 pad 8: Net-(U3-VIN) -> /Supply/DCDC_IN
- U9 pad 30: unconnected-(U9-AOUTB2--Pad30) -> /Codec/AOUTB-
- U9 pad 31: unconnected-(U9-AOUTB2+-Pad31) -> /Codec/AOUTB+
- U9 pad 32: unconnected-(U9-AOUTA2+-Pad32) -> /Codec/AOUTA+
- U9 pad 33: unconnected-(U9-AOUTA2--Pad33) -> /Codec/AOUTA-
- U9 pad 34: /Codec/AOUTB1- -> unconnected-(U9-AOUTB1--Pad34)
- U9 pad 35: /Codec/AOUTB1+ -> unconnected-(U9-AOUTB1+-Pad35)
- U9 pad 36: /Codec/AOUTA1+ -> unconnected-(U9-AOUTA1+-Pad36)
- U9 pad 37: /Codec/AOUTA1- -> unconnected-(U9-AOUTA1--Pad37)
- U9 pad 38: /Codec/MUTEC_0 -> /Amplifier/MUTEC
- U9 pad 4: Net-(C34-Pad1) -> +5V
- U9 pad 41: Net-(U9-VARX) -> +5VA
- U9 pad 51: Net-(C49-Pad1) -> +5V
- U9 pad 7: /Codec/SCL_1 -> /Amplifier/SCL_1
- U9 pad 8: /Codec/SDA_1 -> /Amplifier/SDA_1
Routing:
- net +5V5: track 0.00 -> 134.5 mm, vias 0 -> 2
- net +5V: track 0.00 -> 93.2 mm, vias 0 -> 19
- net GND: track 0.00 -> 84.5 mm, vias 0 -> 355
- net GND2: track 0.00 -> 60.7 mm, vias 0 -> 9
- net /Amplifier/HP_R_0: track 0.00 -> 32.1 mm
- net +5VA: track 0.00 -> 29.1 mm, vias 0 -> 43
- net OP_VCC-: track 0.00 -> 28.5 mm, vias 0 -> 20
- net +3V3: track 0.02 -> 26.5 mm, vias 0 -> 42
- net /Amplifier/HP_L_0: track 0.00 -> 24.2 mm
- net /Supply/DCDC_IN: track 0.00 -> 19.0 mm, vias 0 -> 2
- net Net-(U2-V+): track 0.00 -> 15.9 mm
- net Net-(U5-FEEDBACK): track 0.00 -> 15.5 mm
- net Net-(U5-OUT): track 0.00 -> 11.6 mm
- net Net-(X1-Tri-State): track 0.00 -> 10.3 mm, vias 0 -> 2
- net Net-(U2-FC): track 0.00 -> 8.47 mm, vias 0 -> 2
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- added copper zone on F.Cu, net +3V3
- added copper zone on In2.Cu, net +3V3
- added copper zone on F.Cu, net +5V
- added copper zone on In2.Cu, net +5V
- added copper zone on F.Cu, net +5V5
- added copper zone on F.Cu, net +5VA
- added copper zone on In2.Cu, net +5VA
- added copper zone on F.Cu, net /Input/OPT_VCC
- added copper zone on F.Cu, net /Supply/DCDC_IN
- added copper zone on F.Cu, net /Supply/DCDC_SW
- added copper zone on B.Cu, net GND
- added copper zone on F.Cu, net GND
- added copper zone on In1.Cu, net GND
- added copper zone on F.Cu, net GND2
- added copper zone on In1.Cu, net GND2
- added copper zone on B.Cu, net OP_VCC-
- added copper zone on F.Cu, net OP_VCC-
- added copper zone on F.Cu, net VIN
Other:
- outline, holes or cut-outs redrawn
- board text added: "allow 2.2mm on the sides for sliding slot"

Commit message: backup commit
Parts:
- removed H2, H3: MountingHole, MountingHole:MountingHole_3.2mm_M3
- removed J10: Conn_01x03, Connector_PinHeader_2.54mm:PinHeader_1x03_P2.54mm_Vertical
- moved H1 143.8 mm to (194.3, 53.5)
- moved R49 16.2 mm to (163.5, 121.3), turned to 180 degrees
- moved D2 15.5 mm to (169.3, 125.7)
- moved R48 15.5 mm to (171.2, 125.7)
- moved R50 14.2 mm to (163.5, 119.6), turned to 180 degrees
- moved R44 9.99 mm to (149.7, 127.1)
- moved Q3 8.99 mm to (153.8, 127.1), turned to -90 degrees
- moved R74 8.45 mm to (141.7, 88.6)
- moved J4 7.60 mm to (181.7, 125.3), turned to 90 degrees
- moved C81 7.19 mm to (178.8, 124.9), turned to 90 degrees
- moved R40 6.77 mm to (151.2, 127.1), turned to -90 degrees
- moved R51 5.78 mm to (163.5, 117.9)
- moved R43 5.04 mm to (149.6, 123.2)
- moved R75 3.75 mm to (131.5, 97.6)
- moved R39 2.96 mm to (151.2, 123.2), turned to -90 degrees
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Routing:
- net GND: track 84.5 -> 203.1 mm, vias 355 -> 489
- net /Control/POT_VOLTAGE: track 0.00 -> 59.5 mm, vias 0 -> 1
- net /Amplifier/SCL_1: track 0.00 -> 57.6 mm, vias 0 -> 1
- net /Amplifier/SDA_1: track 0.00 -> 43.4 mm, vias 0 -> 1
- net /Input/SPDIF_DATA: track 0.00 -> 34.5 mm
- net /Amplifier/HP_R_0: track 32.1 -> 0.00 mm
- net Net-(Q3-D): track 0.00 -> 30.9 mm, vias 0 -> 2
- net Net-(Q2-D): track 0.00 -> 29.5 mm, vias 0 -> 2
- net GND2: track 60.7 -> 32.9 mm, vias 9 -> 19
- net VIN: track 0.00 -> 27.0 mm
- net /Microcontroller/ESP32_BOOT: track 0.00 -> 24.9 mm, vias 0 -> 2
- net /Amplifier/HP_L_0: track 24.2 -> 0.00 mm
- net /Codec/AOUTA+: track 0.00 -> 20.3 mm
- net /Codec/AOUTA-: track 0.00 -> 20.2 mm, vias 0 -> 2
- net +3V3: track 26.5 -> 45.9 mm, vias 42 -> 50
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- added copper zone on In2.Cu, net GND
