File: src/hardware/pcb/ample/kicad/ample.kicad_pcb (KiCad board)
At the start: 4 copper layers, 100 x 80 mm, 217 parts, among them J1 DCJ200-05-A, J2 Conn_01x02, J3 NRJ6HM-1-PRE, J4 Conn_02x03_Counter_Clockwise, J5 Conn_01x03, J6 Conn_01x03, J7 Conn_01x03, J8 Conn_01x03, J9 Conn_02x03_Odd_Even, Q1 BSN20, Q2 BSN20, Q3 BSN20, U1 LDL212DR, U10 TSDP11XX, U11 ESP32-WROVER, U12 OPA1632DGN, U13 OPA1632DGN, U2 MAX660MX, U3 RT7272A, U4 LDL212DR, U5 LP2951-5.0_SOIC, U6 LDL212DR, U7 TORX1350A(F), U8 74AHCT1G126, U9 CS42528, X1 ECS-2520MV-xxx-xx

Commit message: backport 1 for rev 00.01
Routing:
- net GND: track 250.7 -> 235.9 mm, vias 590 -> 606
