File: src/hardware/pcb/ample/kicad/amplifier.kicad_sch (KiCad schematic)
At the start: 2 parts, among them U5 MAX13331

Commit message: rev 00.01 schematics almost done
Parts:
- removed J?: AudioJack3, symbol ample-rescue:AudioJack3-Connector
- removed U5: MAX13331, Package_SO:QSOP-16_3.9x4.9mm_P0.635mm, symbol LNIC_Amplifier_Audio:MAX13331
- added C47, C76, C78, C79, C84: 10u, symbol Device:C_Small
- added C77, C80: 100n, symbol Device:C_Small
- added C81, C82, C83: 4u7, symbol Device:C_Small
- added J?: AudioJack3, symbol ample-rescue:AudioJack3-Connector
- added Q1, Q2, Q3: BSN20, Package_TO_SOT_SMD:SOT-23, symbol Transistor_FET:BSN20
- added R47, R52, R53, R68: 10k, symbol Device:R_Small
- added R48, R49, R69: 0R, symbol Device:R_Small
- added R50, R51: np/0R, symbol Device:R_Small
- added TP2, TP3, TP4, TP6, TP7, TP8, TP9: TestPoint, symbol Connector:TestPoint
- added U10: TSDP11XX, Package_DFN_QFN:QFN-20-1EP_4x4mm_P0.5mm_EP2.5x2.5mm, symbol LNIC_Amplifier_Audio:TSDP11XX
Connections:
- new net: J?.R, R48.1
- new net: R48.2, U10.8 (HP_R)
- new net: C84.1, TP2.1, U10.14 (VREG)
- new net: Q2.3 (D), R50.2, R53.1, TP7.1, U10.19 (I2C_SCL)
- new net: C81.2, U10.10 (CPN)
- new net: J?.S, U10.11 (CP_GND)
- new net: C83.1, TP3.1, U10.12 (V+)
- new net: C81.1, U10.13 (CPP)
- new net: Q1.3 (D), R51.2, R52.1, TP6.1, U10.20 (I2C_SDA)
- new net: R49.2, U10.7 (HP_L)
- new net: C82.1, TP4.1, U10.9 (V-)
- new net: J?.T, R49.1
- new net: Q3.3 (D), R69.2
- new net +3V3: Q1.1 (G), Q2.1 (G)
- new net +5V: R52.2, R53.2
- new net +5VA: C47.1, C76.1, C77.1, C78.1, C79.1, C80.1, R47.2, U10.15 (VDDA), U10.18 (VDDA)
- new net AMP_EN: R47.1, R69.1, U10.1 (~{SD})
- new net FILT_LEFT_N: U10.6 (LEFT_IN_N)
- new net FILT_LEFT_P: U10.5 (LEFT_IN_P)
- new net FILT_RIGHT_N: U10.4 (RIGHT_IN_N)
- new net FILT_RIGHT_P: U10.3 (RIGHT_IN_P)
- new net GND: C47.2, C76.2, C77.2, C78.2, C79.2, C80.2, C82.2, C83.2, C84.2, Q3.2 (S), R68.1, U10.16 (GND), U10.17 (GND), U10.2 (GND), U10.21 (PAD)
- new net MUTEC: Q3.1 (G), R68.2
- new net SCL: Q2.2 (S), R50.1, TP9.1
- new net SDA: Q1.2 (S), R51.1, TP8.1
Other:
- note added: "Headphone Amplifier"
- note added: "Level Shifter, might not be needed https://cdn-shop.adafruit.com/datasheets/an97055.pdf"

Commit message: finishing schematics
Parts:
- removed C76: 10u, symbol Device:C_Small
- added C75: 10u, Capacitor_SMD:C_0603_1608Metric, symbol Device:C_Small
- added J6: Conn_01x03, Connector_PinHeader_2.54mm:PinHeader_1x03_P2.54mm_Vertical, symbol Connector_Generic:Conn_01x03
- added L? (x2): ASPI-6045T-220M-T, LNIC_Inductor_SMD:L_Abracon_ASPI-6045T, symbol Device:L_Small
- C68: renamed from C78; footprint (none) -> Capacitor_SMD:C_0603_1608Metric
- C69: renamed from C81; footprint (none) -> Capacitor_SMD:C_0603_1608Metric
- C70: renamed from C79; footprint (none) -> Capacitor_SMD:C_0603_1608Metric
- C71: renamed from C80; footprint (none) -> Capacitor_SMD:C_0603_1608Metric
- C72: renamed from C47; value 10u -> 100n; footprint (none) -> Capacitor_SMD:C_0603_1608Metric
- C73: renamed from C77; value 100n -> 10u; footprint (none) -> Capacitor_SMD:C_0603_1608Metric
- C74: renamed from C82; footprint (none) -> Capacitor_SMD:C_0603_1608Metric
- C76: renamed from C83; footprint (none) -> Capacitor_SMD:C_0603_1608Metric
- C77: renamed from C84; footprint (none) -> Capacitor_SMD:C_0603_1608Metric
- R38: renamed from R68; footprint (none) -> Resistor_SMD:R_0603_1608Metric
- R39: renamed from R51; footprint (none) -> Resistor_SMD:R_0603_1608Metric
- R40: renamed from R50; footprint (none) -> Resistor_SMD:R_0603_1608Metric
- R41: renamed from R47; footprint (none) -> Resistor_SMD:R_0603_1608Metric
- R42: renamed from R69; footprint (none) -> Resistor_SMD:R_0603_1608Metric
- R43: renamed from R52; footprint (none) -> Resistor_SMD:R_0603_1608Metric
- R44: renamed from R53; footprint (none) -> Resistor_SMD:R_0603_1608Metric
- R45: renamed from R49; footprint (none) -> Resistor_SMD:R_0603_1608Metric
- R46: renamed from R48; footprint (none) -> Resistor_SMD:R_0603_1608Metric
- TP10: renamed from TP4; footprint (none) -> TestPoint:TestPoint_Pad_D2.0mm
- TP11: renamed from TP3; footprint (none) -> TestPoint:TestPoint_Pad_D2.0mm
- TP12: renamed from TP2; footprint (none) -> TestPoint:TestPoint_Pad_D2.0mm
- TP6: renamed from TP8; footprint (none) -> TestPoint:TestPoint_Pad_D2.0mm
- TP7: renamed from TP9; footprint (none) -> TestPoint:TestPoint_Pad_D2.0mm
- TP8: renamed from TP6; footprint (none) -> TestPoint:TestPoint_Pad_D2.0mm
- TP9: renamed from TP7; footprint (none) -> TestPoint:TestPoint_Pad_D2.0mm
- renumbered Q3 to Q1, Q1 to Q2, Q2 to Q3
Connections:
- net +5VA: now also C75.1, L?.1, L?.2; no longer C70.1, C71.1, C72.1, C73.1, U10.15 (VDDA), U10.18 (VDDA)
- net GND: now also C75.2
- net at J?.R, R46.1: now also J6.2 (Pin_2)
- net at J?.T, R45.1: now also J6.1 (Pin_1)
- new net: C72.1, C73.1, L?.1, U10.18 (VDDA)
- new net: C70.1, C71.1, L?.2, U10.15 (VDDA)
Other:
- note added: "maybe reduce to 1 inductor"
- moved on the sheet: C68, C73

Commit message: layout init
Parts:
- removed C70: 10u, Capacitor_SMD:C_0603_1608Metric, symbol Device:C_Small
- removed J?: AudioJack3, symbol ample-rescue:AudioJack3-Connector
- removed L? (x2): ASPI-6045T-220M-T, LNIC_Inductor_SMD:L_Abracon_ASPI-6045T, symbol Device:L_Small
- removed R45, R46: 0R, Resistor_SMD:R_0603_1608Metric, symbol Device:R_Small
- removed TP10, TP11, TP12: TestPoint, TestPoint:TestPoint_Pad_D2.0mm, symbol Connector:TestPoint
- added C102, C103: 10u, Capacitor_SMD:C_0603_1608Metric, symbol Device:C_Small
- added J11: NRJ6HM-1-PRE, LNIC_Connector_Audio:Jack_6.35mm_Neutrik_NRJ6HM-1-PRE_Horizontal, symbol Connector_Audio:NRJ6HM-1-PRE
Connections:
- net +5VA: now also C71.1, C72.1, C73.1, U10.15 (VDDA), U10.18 (VDDA), C102.1, C103.1
- net GND: now also C102.2, C103.2; no longer C74.2, C76.2, C77.2
- net HP_R_0: now reaches J6.2 (Pin_2)
- net HP_R_0: now also U10.8 (HP_R), J11.R
- net GND2: now reaches U10.11 (CP_GND)
- net GND2: now also C74.2, C76.2, C77.2, J6.3 (Pin_3), J11.S
- net HP_L_0: now reaches U10.7 (HP_L)
- net HP_L_0: now also J6.1 (Pin_1), J11.T
- net SCL renamed SCL_1
- net SDA renamed SDA_1
- no-connect marks 0 -> 2
Other:
- note added: "change mute polarity in register to active high for this to work"
- moved on the sheet: C68, C74, C75, C76, C77, J6

Commit message: backup commit
Parts:
- removed J6: Conn_01x03, Connector_PinHeader_2.54mm:PinHeader_1x03_P2.54mm_Vertical, symbol Connector_Generic:Conn_01x03
Changed lines of the file:
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@@
   (junction (at 80.01 60.96) (diameter 0) (color 0 0 0 0)
   )
-  (junction (at 236.22 66.04) (diameter 0) (color 0 0 0 0)
-  )
-  (junction (at 231.14 71.12) (diameter 0) (color 0 0 0 0)
-  )
   (junction (at 71.12 120.65) (diameter 0) (color 0 0 0 0)
   )
@@
   )
   (junction (at 80.01 85.09) (diameter 0) (color 0 0 0 0)
-  )
-  (junction (at 233.68 68.58) (diameter 0) (color 0 0 0 0)
   )
   (no_connect (at 247.65 63.5))
@@
     (stroke (width 0) (type default))
   )
-  (wire (pts (xy 176.53 66.04) (xy 236.22 66.04))
-    (stroke (width 0) (type default))
-  )
   (wire (pts (xy 68.58 76.2) (xy 60.96 76.2))
     (stroke (width 0) (type default))
@@
     (stroke (width 0) (type default))
   )
-  (wire (pts (xy 236.22 66.04) (xy 247.65 66.04))
-    (stroke (width 0) (type default))
-  )
-  (wire (pts (xy 233.68 82.55) (xy 238.76 82.55))
+  (wire (pts (xy 176.53 66.04) (xy 247.65 66.04))
     (stroke (width 0) (type default))
   )
@@
     (stroke (width 0) (type default))
   )
-  (wire (pts (xy 238.76 80.01) (xy 236.22 80.01))
-    (stroke (width 0) (type default))
-  )
   (wire (pts (xy 187.96 44.45) (xy 187.96 46.99))
     (stroke (width 0) (type default))
@@
     (stroke (width 0) (type default))
   )
-  (wire (pts (xy 185.42 71.12) (xy 231.14 71.12))
-    (stroke (width 0) (type default))
-  )
   (wire (pts (xy 243.84 71.12) (xy 243.84 68.58))
     (stroke (width 0) (type default))
@@
     (stroke (width 0) (type default))
   )
-  (wire (pts (xy 238.76 85.09) (xy 231.14 85.09))
-    (stroke (width 0) (type default))
-  )
   (wire (pts (xy 203.2 111.76) (xy 203.2 109.22))
     (stroke (width 0) (type default))
@@
     (stroke (width 0) (type default))
   )
-  (wire (pts (xy 176.53 68.58) (xy 233.68 68.58))
+  (wire (pts (xy 176.53 68.58) (xy 243.84 68.58))
     (stroke (width 0) (type default))
   )
@@
     (stroke (width 0) (type default))
   )
-  (wire (pts (xy 233.68 68.58) (xy 233.68 82.55))
-    (stroke (width 0) (type default))
-  )
   (wire (pts (xy 80.01 85.09) (xy 91.44 85.09))
     (stroke (width 0) (type default))
@@
     (stroke (width 0) (type default))
   )
-  (wire (pts (xy 233.68 68.58) (xy 243.84 68.58))
-    (stroke (width 0) (type default))
-  )
   (wire (pts (xy 199.39 44.45) (xy 199.39 46.99))
     (stroke (width 0) (type default))
@@
     (stroke (width 0) (type default))
   )
-  (wire (pts (xy 231.14 71.12) (xy 242.57 71.12))
-    (stroke (width 0) (type default))
-  )
-  (wire (pts (xy 236.22 80.01) (xy 236.22 66.04))
+  (wire (pts (xy 185.42 71.12) (xy 242.57 71.12))
     (stroke (width 0) (type default))
   )
@@
   )
   (wire (pts (xy 167.64 36.83) (xy 176.53 36.83))
-    (stroke (width 0) (type default))
-  )
-  (wire (pts (xy 231.14 85.09) (xy 231.14 71.12))
     (stroke (width 0) (type default))
   )
@@
         )
       )
-    )
-  )
-  (symbol (lib_id "Connector_Generic:Conn_01x03") (at 243.84 82.55 0) (unit 1)
-    (in_bom yes) (on_board yes) (dnp no)
-    (property "Reference" "J6" (at 245.872 81.4832 0)
-      (effects (font (size 1.27 1.27)) (justify left))
-    )
-    (property "Value" "Conn_01x03" (at 245.872 83.7946 0)
-      (effects (font (size 1.27 1.27)) (justify left))
-    )
-    (property "Footprint" "Connector_PinHeader_2.54mm:PinHeader_1x03_P2.54mm_Vertical" (at 243.84 82.55 0)
-      (effects (font (size 1.27 1.27)) hide)
-    )
-    (property "Datasheet" "~" (at 243.84 82.55 0)
-      (effects (font (size 1.27 1.27)) hide)
-    )
-    (pin "1")
-    (pin "2")
-    (pin "3")
-    (instances
-      (project "ample"
-        (path "/bb5c9149-9eb8-4a9c-8d50-f58c12224ad5/00000000-0000-0000-0000-0000628f8524"
-          (reference "J6") (unit 1)
-        )
-        (path "/bb5c9149-9eb8-4a9c-8d50-f58c12224ad5/00000000-0000-0000-0000-0000628f85ad"
-          (reference "J10") (unit 1)
-        )
-      )

Commit message: rev 00.01
Parts:
- renumbered C68 to C75, C102 to C76, C69 to C77, C71 to C78, C72 to C79, C73 to C80, C74 to C81, C103 to C82, C76 to C83, C75 to C84, C77 to C85, J11 to J3, R38 to R34, R39 to R35, R40 to R36, R41 to R37, R42 to R38, R43 to R39, R44 to R40, TP6 to TP19, TP7 to TP20, TP8 to TP21, TP9 to TP22

Commit message: rev 00.01
Parts:
- removed TP19, TP20, TP21, TP22: TestPoint, TestPoint:TestPoint_Pad_D2.0mm, symbol Connector:TestPoint
Changed lines of the file:
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@@
   (junction (at 91.44 60.96) (diameter 0) (color 0 0 0 0)
   )
-  (junction (at 104.14 68.58) (diameter 0) (color 0 0 0 0)
-  )
   (junction (at 167.64 36.83) (diameter 0) (color 0 0 0 0)
   )
@@
   (junction (at 185.42 71.12) (diameter 0) (color 0 0 0 0)
   )
-  (junction (at 48.26 60.96) (diameter 0) (color 0 0 0 0)
-  )
   (junction (at 59.69 135.89) (diameter 0) (color 0 0 0 0)
   )
@@
   (junction (at 176.53 46.99) (diameter 0) (color 0 0 0 0)
   )
-  (junction (at 48.26 85.09) (diameter 0) (color 0 0 0 0)
-  )
   (junction (at 187.96 36.83) (diameter 0) (color 0 0 0 0)
   )
@@
   )
   (junction (at 158.75 114.3) (diameter 0) (color 0 0 0 0)
-  )
-  (junction (at 104.14 71.12) (diameter 0) (color 0 0 0 0)
   )
   (junction (at 60.96 60.96) (diameter 0) (color 0 0 0 0)
@@
     (stroke (width 0) (type default))
   )
-  (wire (pts (xy 43.18 60.96) (xy 48.26 60.96))
+  (wire (pts (xy 43.18 60.96) (xy 60.96 60.96))
     (stroke (width 0) (type default))
   )
@@
     (stroke (width 0) (type default))
   )
-  (wire (pts (xy 48.26 60.96) (xy 60.96 60.96))
-    (stroke (width 0) (type default))
-  )
   (wire (pts (xy 156.21 36.83) (xy 156.21 58.42))
     (stroke (width 0) (type default))
@@
     (stroke (width 0) (type default))
   )
-  (wire (pts (xy 48.26 85.09) (xy 43.18 85.09))
-    (stroke (width 0) (type default))
-  )
   (wire (pts (xy 199.39 36.83) (xy 199.39 39.37))
     (stroke (width 0) (type default))
   )
-  (wire (pts (xy 104.14 71.12) (xy 140.97 71.12))
-    (stroke (width 0) (type default))
-  )
   (wire (pts (xy 158.75 114.3) (xy 158.75 115.57))
     (stroke (width 0) (type default))
@@
     (stroke (width 0) (type default))
   )
-  (wire (pts (xy 99.06 71.12) (xy 104.14 71.12))
+  (wire (pts (xy 99.06 71.12) (xy 140.97 71.12))
     (stroke (width 0) (type default))
   )
@@
     (stroke (width 0) (type default))
   )
-  (wire (pts (xy 99.06 68.58) (xy 104.14 68.58))
+  (wire (pts (xy 99.06 68.58) (xy 140.97 68.58))
     (stroke (width 0) (type default))
   )
@@
     (stroke (width 0) (type default))
   )
-  (wire (pts (xy 60.96 85.09) (xy 48.26 85.09))
+  (wire (pts (xy 43.18 85.09) (xy 60.96 85.09))
     (stroke (width 0) (type default))
   )
@@
   )
   (wire (pts (xy 116.84 48.26) (xy 116.84 46.99))
-    (stroke (width 0) (type default))
-  )
-  (wire (pts (xy 104.14 68.58) (xy 140.97 68.58))
     (stroke (width 0) (type default))
   )
@@
   (hierarchical_label "FILT_RIGHT_P" (shape input) (at 135.89 77.47 180) (fields_autoplaced)
     (effects (font (size 1.27 1.27)) (justify right))
-  )
-  (symbol (lib_id "Connector:TestPoint") (at 104.14 71.12 180) (unit 1)
-    (in_bom yes) (on_board yes) (dnp no) (fields_autoplaced)
-    (property "Reference" "TP22" (at 106.68 73.152 0)
-      (effects (font (size 1.27 1.27)) (justify right))
-    )
-    (property "Value" "TestPoint" (at 106.68 75.692 0)
-      (effects (font (size 1.27 1.27)) (justify right))
-    )
-    (property "Footprint" "TestPoint:TestPoint_Pad_D2.0mm" (at 99.06 71.12 0)
-      (effects (font (size 1.27 1.27)) hide)
-    )
-    (property "Datasheet" "~" (at 99.06 71.12 0)
-      (effects (font (size 1.27 1.27)) hide)
-    )
-    (pin "1")
-    (instances
-      (project "ample"
-        (path "/bb5c9149-9eb8-4a9c-8d50-f58c12224ad5/00000000-0000-0000-0000-0000628f85ad"
-          (reference "TP22") (unit 1)
-        )
-      )
-    )
   )
   (symbol (lib_id "power:+5V") (at 91.44 48.26 0) (unit 1)
@@
     )
   )
-  (symbol (lib_id "Connector:TestPoint") (at 48.26 60.96 0) (unit 1)
-    (in_bom yes) (on_board yes) (dnp no) (fields_autoplaced)
-    (property "Reference" "TP19" (at 50.8 56.388 0)
-      (effects (font (size 1.27 1.27)) (justify left))
-    )
-    (property "Value" "TestPoint" (at 50.8 58.928 0)
-      (effects (font (size 1.27 1.27)) (justify left))
-    )
-    (property "Footprint" "TestPoint:TestPoint_Pad_D2.0mm" (at 53.34 60.96 0)
-      (effects (font (size 1.27 1.27)) hide)
-    )
-    (property "Datasheet" "~" (at 53.34 60.96 0)
-      (effects (font (size 1.27 1.27)) hide)
-    )
-    (pin "1")
-    (instances
-      (project "ample"
-        (path "/bb5c9149-9eb8-4a9c-8d50-f58c12224ad5/00000000-0000-0000-0000-0000628f85ad"
-          (reference "TP19") (unit 1)
-        )
-      )
-    )
-  )
   (symbol (lib_id "Device:C_Small") (at 147.32 41.91 0) (unit 1)
     (in_bom yes) (on_board yes) (dnp no) (fields_autoplaced)
@@
     )
   )
-  (symbol (lib_id "Connector:TestPoint") (at 104.14 68.58 0) (unit 1)
-    (in_bom yes) (on_board yes) (dnp no) (fields_autoplaced)
-    (property "Reference" "TP21" (at 106.68 64.008 0)
-      (effects (font (size 1.27 1.27)) (justify left))
-    )
-    (property "Value" "TestPoint" (at 106.68 66.548 0)
-      (effects (font (size 1.27 1.27)) (justify left))
-    )
-    (property "Footprint" "TestPoint:TestPoint_Pad_D2.0mm" (at 109.22 68.58 0)
-      (effects (font (size 1.27 1.27)) hide)
-    )
-    (property "Datasheet" "~" (at 109.22 68.58 0)
-      (effects (font (size 1.27 1.27)) hide)
-    )
-    (pin "1")
-    (instances
-      (project "ample"
-        (path "/bb5c9149-9eb8-4a9c-8d50-f58c12224ad5/00000000-0000-0000-0000-0000628f85ad"
-          (reference "TP21") (unit 1)
-        )
-      )
-    )
-  )
   (symbol (lib_id "power:GND") (at 158.75 115.57 0) (unit 1)
     (in_bom yes) (on_board yes) (dnp no)
@@
         )
       )
-    )
-  )
-  (symbol (lib_id "Connector:TestPoint") (at 48.26 85.09 0) (unit 1)
-    (in_bom yes) (on_board yes) (dnp no) (fields_autoplaced)
-    (property "Reference" "TP20" (at 50.8 80.518 0)
-      (effects (font (size 1.27 1.27)) (justify left))
-    )
-    (property "Value" "TestPoint" (at 50.8 83.058 0)
-      (effects (font (size 1.27 1.27)) (justify left))
-    )
-    (property "Footprint" "TestPoint:TestPoint_Pad_D2.0mm" (at 53.34 85.09 0)
-      (effects (font (size 1.27 1.27)) hide)
-    )
-    (property "Datasheet" "~" (at 53.34 85.09 0)
-      (effects (font (size 1.27 1.27)) hide)
-    )
-    (pin "1")
-    (instances
-      (project "ample"
-        (path "/bb5c9149-9eb8-4a9c-8d50-f58c12224ad5/00000000-0000-0000-0000-0000628f85ad"
-          (reference "TP20") (unit 1)
-        )
-      )

Commit message: backport 1 for rev 00.01
Other:
- title: (none) -> ample/Amplifier
Changed lines of the file:
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@@
 (kicad_sch (version 20230121) (generator eeschema)
   (paper "A4")
+  (title_block
+    (title "ample/Amplifier")
+    (date "2023-07-14")
+    (rev "00.01")
+  )
   (junction (at 91.44 60.96) (diameter 0) (color 0 0 0 0)
   )
