File: src/hardware/pcb/ample/kicad/codec.kicad_sch (KiCad schematic)
At the start: 51 parts, among them U11 CS42528, X1 ECS-2520MV-xxx-xx

Commit message: rev 00.01 schematics almost done
Parts:
- added C46: 10u, symbol Device:C_Small
- C30, C31, C60: value 100n -> 2u2
- C71: value 1u -> 2u2
- C72: value 1u -> 10u
Connections:
- net +3V3: now also C46.1
- net GND: now also C46.2
- net CS42528_INT renamed CODEC_INT
- net CS42528_nRST renamed CODEC_nRST
- net SAI_LRCLK: no longer names the net of U11.60 (SAI_LRCK)
- net SAI_SCLK: no longer names the net of U11.61 (SAI_SCLK)
- no-connect marks 24 -> 26
Other:
- note added: "for review: Go over all pins in datasheet"

Commit message: finishing schematics
Parts:
- removed L3 (x3): 22u, symbol Device:L_Small
- added L? (x2): ASPI-6045T-220M-T, LNIC_Inductor_SMD:L_Abracon_ASPI-6045T, symbol Device:L_Small
- added TP8 (x4): TestPoint, TestPoint:TestPoint_Pad_D2.0mm, symbol Connector:TestPoint
- C32: renamed from C29; value C_Small -> 100n; footprint (none) -> Capacitor_SMD:C_0603_1608Metric
- C33: renamed from C30; footprint (none) -> Capacitor_SMD:C_0603_1608Metric
- C34: renamed from C31; footprint (none) -> Capacitor_SMD:C_0603_1608Metric
- C35: renamed from C72; footprint (none) -> Capacitor_SMD:C_0603_1608Metric
- C36: renamed from C73; footprint (none) -> Capacitor_SMD:C_0603_1608Metric
- C37: renamed from C61; footprint (none) -> Capacitor_SMD:C_0603_1608Metric
- C38: renamed from C60; footprint (none) -> Capacitor_SMD:C_0603_1608Metric
- C39: renamed from C32; footprint (none) -> Capacitor_SMD:C_0603_1608Metric
- C40: renamed from C71; footprint (none) -> Capacitor_SMD:C_0603_1608Metric
- C41: renamed from C33; footprint (none) -> Capacitor_SMD:C_0603_1608Metric
- C42: renamed from C70; footprint (none) -> Capacitor_SMD:C_0603_1608Metric
- C43: renamed from C69; footprint (none) -> Capacitor_SMD:C_0603_1608Metric
- C44: renamed from C68; footprint Capacitor_THT:CP_Radial_Tantal_D8.0mm_P5.00mm -> Capacitor_THT:CP_Radial_D6.3mm_P2.50mm
- C45: renamed from C62; footprint (none) -> Capacitor_SMD:C_0603_1608Metric
- C46: renamed from C34; footprint (none) -> Capacitor_SMD:C_0603_1608Metric
- C47: renamed from C35; footprint (none) -> Capacitor_SMD:C_0603_1608Metric
- C48: renamed from C36; footprint (none) -> Capacitor_SMD:C_0603_1608Metric
- C49: renamed from C37; footprint (none) -> Capacitor_SMD:C_0603_1608Metric
- C50: renamed from C66; footprint (none) -> Capacitor_SMD:C_0603_1608Metric
- C51: renamed from C38; footprint (none) -> Capacitor_SMD:C_0603_1608Metric
- C52: renamed from C39; footprint (none) -> Capacitor_SMD:C_0603_1608Metric
- C53: renamed from C46; footprint (none) -> Capacitor_SMD:C_0603_1608Metric
- C54: renamed from C40; footprint (none) -> Capacitor_SMD:C_0603_1608Metric
- C55: renamed from C41; footprint (none) -> Capacitor_SMD:C_0603_1608Metric
- C56: renamed from C42; footprint (none) -> Capacitor_SMD:C_0603_1608Metric
- C57: renamed from C26; footprint (none) -> Capacitor_SMD:C_0603_1608Metric
- C58: renamed from C54; footprint (none) -> Capacitor_SMD:C_0603_1608Metric
- C59: renamed from C55; footprint (none) -> Capacitor_SMD:C_0603_1608Metric
- C60: renamed from C56; footprint (none) -> Capacitor_SMD:C_0603_1608Metric
- C61: renamed from C57; footprint (none) -> Capacitor_SMD:C_0603_1608Metric
- C62: renamed from C58; footprint (none) -> Capacitor_SMD:C_0603_1608Metric
- C63: renamed from C59; footprint (none) -> Capacitor_SMD:C_0603_1608Metric
- C64: renamed from C43; footprint (none) -> Capacitor_SMD:C_0603_1608Metric
- C65: renamed from C67; footprint (none) -> Capacitor_SMD:C_0603_1608Metric
- C66: renamed from C65; footprint (none) -> Capacitor_SMD:C_0603_1608Metric
- C67: renamed from C64; footprint (none) -> Capacitor_SMD:C_0603_1608Metric
- L?: renamed from L3; value 22u -> ASPI-6045T-220M-T; footprint (none) -> LNIC_Inductor_SMD:L_Abracon_ASPI-6045T
- R29: renamed from R21; footprint (none) -> Resistor_SMD:R_0603_1608Metric
- R30: renamed from R19; footprint (none) -> Resistor_SMD:R_0603_1608Metric
- R31: renamed from R20; footprint (none) -> Resistor_SMD:R_0603_1608Metric
- R32: renamed from R17; footprint (none) -> Resistor_SMD:R_0603_1608Metric
- R33: renamed from R22; footprint (none) -> Resistor_SMD:R_0603_1608Metric
- R34: renamed from R23; footprint (none) -> Resistor_SMD:R_0603_1608Metric
- R35: footprint (none) -> Resistor_SMD:R_0603_1608Metric
- R36: renamed from R24; footprint (none) -> Resistor_SMD:R_0603_1608Metric
- R37: renamed from R25; footprint (none) -> Resistor_SMD:R_0603_1608Metric
- TP5: renamed from TP1; footprint (none) -> TestPoint:TestPoint_Pad_D2.0mm
- renumbered U11 to U9
Connections:
- net +3V3: now also C38.1, R30.2, X1.4 (VDD), TP8.1
- net +5V: now also L?.2
- net +5VA: now also L?.2
- net at C34.1, C35.1, C36.1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: now also TP8.1
- net at C55.1, C56.1, C64.1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: now also L?.1, TP8.1
- net at C49.1, C52.1, U9.51 (VD): now also L?.1, TP8.1
Other:
- moved on the sheet: C33, C34, C37

Commit message: layout init
Parts:
- removed C33: 2u2, Capacitor_SMD:C_0603_1608Metric, symbol Device:C_Small
- removed L? (x3): ASPI-6045T-220M-T, LNIC_Inductor_SMD:L_Abracon_ASPI-6045T, symbol Device:L_Small
- removed R36: 0R, Resistor_SMD:R_0603_1608Metric, symbol Device:R_Small
- removed R37: 10k, Resistor_SMD:R_0603_1608Metric, symbol Device:R_Small
- C34: value 2u2 -> 10u
- R31: value 0R -> np/0R
Connections:
- net MUTEC_0 is gone; now on net MUTEC: U9.38 (MUTEC)
- net +5V: now also C34.1, C35.1, C36.1, C49.1, C52.1, TP8.1, TP8.1, U9.4 (VD), U9.51 (VD)
- net +5VA: now also C55.1, C56.1, C64.1, TP8.1, U9.41 (VARX)
- net AOUTB-: now reaches U9.30 (AOUTB2-)
- net AOUTB+: now reaches U9.31 (AOUTB2+)
- net AOUTA+: now reaches U9.32 (AOUTA2+)
- net AOUTA-: now reaches U9.33 (AOUTA2-)
- net AOUTA1+: no longer names the net of U9.36 (AOUTA1+)
- net AOUTA1-: no longer names the net of U9.37 (AOUTA1-)
- net AOUTB1+: no longer names the net of U9.35 (AOUTB1+)
- net AOUTB1-: no longer names the net of U9.34 (AOUTB1-)
Other:
- moved on the sheet: C54, C65

Commit message: rev 00.01
Parts:
- removed C62, C63: 100n, Capacitor_SMD:C_0603_1608Metric, symbol Device:C_Small
- renumbered C32 to C42, C34 to C43, C35 to C44, C36 to C45, C37 to C46, C38 to C47, C39 to C48, C40 to C49, C41 to C50, C42 to C51, C43 to C52, C44 to C53, C45 to C54, C46 to C55, C47 to C56, C48 to C57, C49 to C58, C50 to C59, C51 to C60, C52 to C61, C53 to C62, C54 to C63, C55 to C64, C56 to C65, C57 to C66, C58 to C67, C59 to C68, C60 to C69, C61 to C70, C64 to C71, C65 to C72, C66 to C73, C67 to C74, R29 to R27, R30 to R28, R31 to R29, R32 to R30, R33 to R31, R34 to R32, R35 to R33, TP5 to TP15, TP8 to TP?
Connections:
- no-connect marks 26 -> 28
Other:
- moved on the sheet: C66, C67, C68, C69, C70

Commit message: rev 00.01
Parts:
- removed TP15, TP? (x4): TestPoint, TestPoint:TestPoint_Pad_D2.0mm, symbol Connector:TestPoint
Connections:
- no-connect marks 28 -> 29

Commit message: backport 1 for rev 00.01
Other:
- title: CS42528 -> ample/Codec
Changed lines of the file:
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@@
   (paper "A3")
   (title_block
-    (title "CS42528")
-    (date "2022-06-02")
+    (title "ample/Codec")
+    (date "2023-07-14")
     (rev "00.01")
   )
