File: src/hardware/pcb/ample/kicad/dac_filter.kicad_sch (KiCad schematic)
At the start: 44 parts, among them U5 OPA1632DGN, U6 OPA1632DGN

Commit message: finishing schematics
Parts:
- C84: renamed from C86; footprint (none) -> Capacitor_SMD:C_0603_1608Metric
- C85: renamed from C89; footprint (none) -> Capacitor_SMD:C_0603_1608Metric
- C86: renamed from C88; footprint (none) -> Capacitor_SMD:C_0603_1608Metric
- C87, C92, C93: footprint (none) -> Capacitor_SMD:C_0603_1608Metric
- C88: renamed from C90; footprint (none) -> Capacitor_SMD:C_0603_1608Metric
- C89: renamed from C91; footprint (none) -> Capacitor_SMD:C_0603_1608Metric
- C90: renamed from C52; footprint (none) -> Capacitor_SMD:C_0603_1608Metric
- C91: renamed from C85; footprint (none) -> Capacitor_SMD:C_0603_1608Metric
- C94: renamed from C53; footprint (none) -> Capacitor_SMD:C_0603_1608Metric
- C95: renamed from C94; footprint (none) -> Capacitor_SMD:C_0603_1608Metric
- C96: renamed from C19; footprint (none) -> Capacitor_SMD:C_0603_1608Metric
- C97: renamed from C95; footprint (none) -> Capacitor_SMD:C_0603_1608Metric
- C98: renamed from C21; footprint (none) -> Capacitor_SMD:C_0603_1608Metric
- C99: renamed from C96; footprint (none) -> Capacitor_SMD:C_0603_1608Metric
- R58: renamed from R33; footprint (none) -> Resistor_SMD:R_0603_1608Metric
- R59: renamed from R54; footprint (none) -> Resistor_SMD:R_0603_1608Metric
- R60: renamed from R59; footprint (none) -> Resistor_SMD:R_0603_1608Metric
- R61: renamed from R60; footprint (none) -> Resistor_SMD:R_0603_1608Metric
- R62: renamed from R55; footprint (none) -> Resistor_SMD:R_0603_1608Metric
- R63: renamed from R56; footprint (none) -> Resistor_SMD:R_0603_1608Metric
- R64: renamed from R61; footprint (none) -> Resistor_SMD:R_0603_1608Metric
- R65: renamed from R62; footprint (none) -> Resistor_SMD:R_0603_1608Metric
- R66: renamed from R57; footprint (none) -> Resistor_SMD:R_0603_1608Metric
- R67: renamed from R58; footprint (none) -> Resistor_SMD:R_0603_1608Metric
- R68: renamed from R63; footprint (none) -> Resistor_SMD:R_0603_1608Metric
- R69: renamed from R64; footprint (none) -> Resistor_SMD:R_0603_1608Metric
- R70: renamed from R9; footprint (none) -> Resistor_SMD:R_0603_1608Metric
- R71: renamed from R18; footprint (none) -> Resistor_SMD:R_0603_1608Metric
- R72: renamed from R65; footprint (none) -> Resistor_SMD:R_0603_1608Metric
- R73: renamed from R66; footprint (none) -> Resistor_SMD:R_0603_1608Metric
- R74: renamed from R8; footprint (none) -> Resistor_SMD:R_0603_1608Metric
- R75: renamed from R67; footprint (none) -> Resistor_SMD:R_0603_1608Metric
- TP13: renamed from TP10; footprint (none) -> TestPoint:TestPoint_Pad_D2.0mm
- TP14: renamed from TP11; footprint (none) -> TestPoint:TestPoint_Pad_D2.0mm
- TP15: renamed from TP14; footprint (none) -> TestPoint:TestPoint_Pad_D2.0mm
- TP16: renamed from TP15; footprint (none) -> TestPoint:TestPoint_Pad_D2.0mm
- TP17: renamed from TP12; footprint (none) -> TestPoint:TestPoint_Pad_D2.0mm
- TP18: renamed from TP13; footprint (none) -> TestPoint:TestPoint_Pad_D2.0mm
- TP19: renamed from TP16; footprint (none) -> TestPoint:TestPoint_Pad_D2.0mm
- TP20: renamed from TP17; footprint (none) -> TestPoint:TestPoint_Pad_D2.0mm
- renumbered U5 to U12, U6 to U13

Commit message: layout init
Connections:
- net FILT_LEFT_N: now also C93.2, R73.2, TP20.1; no longer C93.1, R72.2, TP19.1
- net FILT_LEFT_P: now also C93.1, R72.2, TP19.1; no longer C93.2, R73.2, TP20.1
- net FILT_RIGHT_N: now also C91.2, R71.2, TP18.1; no longer C91.1, R70.2, TP17.1
- net FILT_RIGHT_P: now also C91.1, R70.2, TP17.1; no longer C91.2, R71.2, TP18.1
- net AOUTA1+ renamed AOUTA-
- net AOUTA1- renamed AOUTA+
- net AOUTB1+ renamed AOUTB-
- net AOUTB1- renamed AOUTB+
Changed lines of the file:
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@@
     (effects (font (size 1.27 1.27)) (justify left bottom))
   )
-  (hierarchical_label "AOUTA1+" (shape input) (at 54.61 67.31 180) (fields_autoplaced)
+  (hierarchical_label "AOUTA-" (shape input) (at 54.61 67.31 180) (fields_autoplaced)
     (effects (font (size 1.27 1.27)) (justify right))
   )
-  (hierarchical_label "FILT_LEFT_N" (shape output) (at 215.9 137.16 0) (fields_autoplaced)
+  (hierarchical_label "AOUTB+" (shape input) (at 54.61 137.16 180) (fields_autoplaced)
+    (effects (font (size 1.27 1.27)) (justify right))
+  )
+  (hierarchical_label "FILT_LEFT_N" (shape output) (at 215.9 142.24 0) (fields_autoplaced)
     (effects (font (size 1.27 1.27)) (justify left))
   )
-  (hierarchical_label "FILT_LEFT_P" (shape output) (at 215.9 142.24 0) (fields_autoplaced)
+  (hierarchical_label "FILT_RIGHT_N" (shape output) (at 215.9 67.31 0) (fields_autoplaced)
     (effects (font (size 1.27 1.27)) (justify left))
   )
-  (hierarchical_label "AOUTA1-" (shape input) (at 54.61 62.23 180) (fields_autoplaced)
+  (hierarchical_label "AOUTB-" (shape input) (at 54.61 142.24 180) (fields_autoplaced)
     (effects (font (size 1.27 1.27)) (justify right))
   )
-  (hierarchical_label "AOUTB1-" (shape input) (at 54.61 137.16 180) (fields_autoplaced)
+  (hierarchical_label "AOUTA+" (shape input) (at 54.61 62.23 180) (fields_autoplaced)
     (effects (font (size 1.27 1.27)) (justify right))
   )
-  (hierarchical_label "FILT_RIGHT_P" (shape output) (at 215.9 67.31 0) (fields_autoplaced)
+  (hierarchical_label "FILT_LEFT_P" (shape output) (at 215.9 137.16 0) (fields_autoplaced)
     (effects (font (size 1.27 1.27)) (justify left))
   )
-  (hierarchical_label "FILT_RIGHT_N" (shape output) (at 215.9 62.23 0) (fields_autoplaced)
+  (hierarchical_label "FILT_RIGHT_P" (shape output) (at 215.9 62.23 0) (fields_autoplaced)
     (effects (font (size 1.27 1.27)) (justify left))
   )
-  (hierarchical_label "AOUTB1+" (shape input) (at 54.61 142.24 180) (fields_autoplaced)
-    (effects (font (size 1.27 1.27)) (justify right))
-  )
   (symbol (lib_id "Device:C_Small") (at 181.61 114.3 0) (unit 1)

Commit message: rev 00.01
Parts:
- renumbered C92 to C100, C93 to C101, C94 to C102, C95 to C103, C96 to C104, C97 to C105, C98 to C106, C99 to C107, C84 to C92, C85 to C93, C86 to C94, C87 to C95, C88 to C96, C89 to C97, C90 to C98, C91 to C99, R58 to R48, R59 to R49, R60 to R50, R61 to R51, R62 to R52, R63 to R53, R64 to R54, R65 to R55, R66 to R56, R67 to R57, R68 to R58, R69 to R59, R70 to R60, R71 to R61, R72 to R62, R73 to R63, R74 to R64, R75 to R65, TP13 to TP23, TP14 to TP24, TP15 to TP25, TP16 to TP26, TP17 to TP27, TP18 to TP28, TP19 to TP29, TP20 to TP30

Commit message: rev 00.01
Parts:
- removed TP23, TP24, TP25, TP26, TP27, TP28, TP29, TP30: TestPoint, TestPoint:TestPoint_Pad_D2.0mm, symbol Connector:TestPoint

Commit message: backport 1 for rev 00.01
Other:
- title: (none) -> ample/DAC Filter
Changed lines of the file:
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@@
 (kicad_sch (version 20230121) (generator eeschema)
   (paper "A4")
+  (title_block
+    (title "ample/DAC Filter")
+    (date "2023-07-14")
+    (rev "00.01")
+  )
   (junction (at 162.56 67.31) (diameter 0) (color 0 0 0 0)
   )
