File: src/hardware/pcb/ample/kicad/input.kicad_sch (KiCad schematic)
At the start: 9 parts, among them U1 74AHCT1G126, U7 TORX1350A(F)

Commit message: rev 00.01 schematics almost done
Other:
- moved on the sheet: R32, R34
Changed lines of the file:
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@@
     (stroke (width 0) (type default))
   )
-  (wire (pts (xy 161.29 123.19) (xy 181.61 123.19))
+  (wire (pts (xy 162.56 123.19) (xy 181.61 123.19))
     (stroke (width 0) (type default))
   )
@@
     (stroke (width 0) (type default))
   )
-  (wire (pts (xy 156.21 123.19) (xy 138.43 123.19))
+  (wire (pts (xy 157.48 123.19) (xy 138.43 123.19))
     (stroke (width 0) (type default))
   )
@@
     (stroke (width 0) (type default))
   )
-  (wire (pts (xy 162.56 76.2) (xy 162.56 78.74))
+  (wire (pts (xy 162.56 76.2) (xy 162.56 80.01))
     (stroke (width 0) (type default))
   )
@@
     (stroke (width 0) (type default))
   )
+  (wire (pts (xy 99.06 106.68) (xy 99.06 105.41))
+    (stroke (width 0) (type default))
+  )
   (wire (pts (xy 129.54 72.39) (xy 129.54 76.2))
     (stroke (width 0) (type default))
   )
-  (wire (pts (xy 162.56 83.82) (xy 162.56 85.09))
-    (stroke (width 0) (type default))
-  )
   (wire (pts (xy 181.61 95.25) (xy 203.2 95.25))
     (stroke (width 0) (type default))
@@
     (stroke (width 0) (type default))
   )
-  (wire (pts (xy 157.48 107.95) (xy 157.48 105.41))
-    (stroke (width 0) (type default))
-  )
-  (text "Optical\nS/PDIF Input" (at 127 52.07 0)
-    (effects (font (size 2.54 2.54)) (justify left bottom))
+  (wire (pts (xy 157.48 106.68) (xy 157.48 105.41))
+    (stroke (width 0) (type default))
+  )
+  (text "Optical\nS/PDIF Input" (at 80.01 68.58 0)
+    (effects (font (size 2.54 2.54) italic) (justify left bottom))
   )
   (label "SPDIF_DATA_1" (at 118.11 95.25 0) (fields_autoplaced)
@@
     (effects (font (size 1.27 1.27)) (justify left))
   )
-  (symbol (lib_id "power:GND") (at 157.48 107.95 0) (unit 1)
+  (symbol (lib_id "power:GND") (at 157.48 106.68 0) (unit 1)
     (in_bom yes) (on_board yes) (dnp no)
-    (property "Reference" "#PWR0110" (at 157.48 114.3 0)
-      (effects (font (size 1.27 1.27)) hide)
-    )
-    (property "Value" "GND" (at 157.607 112.3442 0)
-      (effects (font (size 1.27 1.27)))
-    )
-    (property "Footprint" "" (at 157.48 107.95 0)
-      (effects (font (size 1.27 1.27)) hide)
-    )
-    (property "Datasheet" "" (at 157.48 107.95 0)
+    (property "Reference" "#PWR0110" (at 157.48 113.03 0)
+      (effects (font (size 1.27 1.27)) hide)
+    )
+    (property "Value" "GND" (at 157.607 111.0742 0)
+      (effects (font (size 1.27 1.27)))
+    )
+    (property "Footprint" "" (at 157.48 106.68 0)
+      (effects (font (size 1.27 1.27)) hide)
+    )
+    (property "Datasheet" "" (at 157.48 106.68 0)
       (effects (font (size 1.27 1.27)) hide)
     )
@@
     )
   )
-  (symbol (lib_id "power:GND") (at 99.06 105.41 0) (unit 1)
+  (symbol (lib_id "power:GND") (at 99.06 106.68 0) (unit 1)
     (in_bom yes) (on_board yes) (dnp no)
-    (property "Reference" "#PWR049" (at 99.06 111.76 0)
-      (effects (font (size 1.27 1.27)) hide)
-    )
-    (property "Value" "GND" (at 99.187 109.8042 0)
-      (effects (font (size 1.27 1.27)))
-    )
-    (property "Footprint" "" (at 99.06 105.41 0)
-      (effects (font (size 1.27 1.27)) hide)
-    )
-    (property "Datasheet" "" (at 99.06 105.41 0)
+    (property "Reference" "#PWR049" (at 99.06 113.03 0)
+      (effects (font (size 1.27 1.27)) hide)
+    )
+    (property "Value" "GND" (at 99.187 111.0742 0)
+      (effects (font (size 1.27 1.27)))
+    )
+    (property "Footprint" "" (at 99.06 106.68 0)
+      (effects (font (size 1.27 1.27)) hide)
+    )
+    (property "Datasheet" "" (at 99.06 106.68 0)
       (effects (font (size 1.27 1.27)) hide)
     )
@@
     )
   )
-  (symbol (lib_id "Device:R_Small") (at 162.56 81.28 180) (unit 1)
+  (symbol (lib_id "Device:R_Small") (at 162.56 82.55 180) (unit 1)
     (in_bom yes) (on_board yes) (dnp no) (fields_autoplaced)
-    (property "Reference" "R34" (at 165.1 80.01 0)
+    (property "Reference" "R34" (at 165.1 81.28 0)
       (effects (font (size 1.27 1.27)) (justify right))
     )
-    (property "Value" "0R" (at 165.1 82.55 0)
+    (property "Value" "0R" (at 165.1 83.82 0)
       (effects (font (size 1.27 1.27)) (justify right))
     )
-    (property "Footprint" "" (at 162.56 81.28 0)
-      (effects (font (size 1.27 1.27)) hide)
-    )
-    (property "Datasheet" "~" (at 162.56 81.28 0)
+    (property "Footprint" "" (at 162.56 82.55 0)
+      (effects (font (size 1.27 1.27)) hide)
+    )
+    (property "Datasheet" "~" (at 162.56 82.55 0)
       (effects (font (size 1.27 1.27)) hide)
     )
@@
     )
   )
-  (symbol (lib_id "Device:R_Small") (at 158.75 123.19 90) (unit 1)
+  (symbol (lib_id "Device:R_Small") (at 160.02 123.19 90) (unit 1)
     (in_bom yes) (on_board yes) (dnp no) (fields_autoplaced)
-    (property "Reference" "R32" (at 158.75 118.11 90)
-      (effects (font (size 1.27 1.27)))
-    )
-    (property "Value" "np/0R" (at 158.75 120.65 90)
-      (effects (font (size 1.27 1.27)))
-    )
-    (property "Footprint" "" (at 158.75 123.19 0)
-      (effects (font (size 1.27 1.27)) hide)
-    )
-    (property "Datasheet" "~" (at 158.75 123.19 0)
-      (effects (font (size 1.27 1.27)) hide)
-    )
+    (property "Reference" "R32" (at 160.02 118.11 90)
+      (effects (font (size 1.27 1.27)))
+    )
+    (property "Value" "np/0R" (at 160.02 120.65 90)
+      (effects (font (size 1.27 1.27)))
+    )
+    (property "Footprint" "" (at 160.02 123.19 0)
+      (effects (font (size 1.27 1.27)) hide)
+    )
+    (property "Datasheet" "~" (at 160.02 123.19 0)
+      (effects (font (size 1.27 1.27)) hide)
+    )

Commit message: finishing schematics
Parts:
- removed L3: 22u, symbol Device:L_Small
- added L?: ASPI-6045T-220M-T, LNIC_Inductor_SMD:L_Abracon_ASPI-6045T, symbol Device:L_Small
- added TP8 (x2): TestPoint, TestPoint:TestPoint_Pad_D2.0mm, symbol Connector:TestPoint
- C? (x4): renamed from C44; footprint (none) -> Capacitor_SMD:C_0603_1608Metric
- R27: renamed from R32; footprint (none) -> Resistor_SMD:R_0603_1608Metric
- R28: renamed from R34; footprint (none) -> Resistor_SMD:R_0603_1608Metric
- renumbered U1 to U?
Connections:
- net +5V: now also L?.2
- net SPDIF_DATA: now also TP8.1
- net at C?.2, U7.3 (VCC): now also L?.1, TP8.1

Commit message: layout init
Connections:
- net OPT_VCC: now reaches C?.2, L?.1, TP8.1, U7.3 (VCC)
Changed lines of the file:
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@@
     (effects (font (size 2.54 2.54) italic) (justify left bottom))
+  )
+  (label "OPT_VCC" (at 100.33 76.2 0) (fields_autoplaced)
+    (effects (font (size 1.27 1.27)) (justify left bottom))
   )
   (label "SPDIF_DATA_1" (at 118.11 95.25 0) (fields_autoplaced)

Commit message: rev 00.01
Parts:
- added C?: 1u, Capacitor_SMD:C_0603_1608Metric, symbol Device:C_Small
- renumbered R27 to R25, R28 to R26, TP8 to TP?
Connections:
- net +5V: now also C?.2
- net GND: now also C?.1

Commit message: rev 00.01
Parts:
- removed TP?: TestPoint, TestPoint:TestPoint_Pad_D2.0mm, symbol Connector:TestPoint
Changed lines of the file:
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@@
   (junction (at 99.06 76.2) (diameter 0) (color 0 0 0 0)
   )
-  (junction (at 181.61 102.87) (diameter 0) (color 0 0 0 0)
-  )
   (junction (at 110.49 76.2) (diameter 0) (color 0 0 0 0)
   )
@@
   (junction (at 149.86 76.2) (diameter 0) (color 0 0 0 0)
   )
-  (wire (pts (xy 181.61 123.19) (xy 181.61 102.87))
+  (wire (pts (xy 181.61 95.25) (xy 181.61 123.19))
     (stroke (width 0) (type default))
   )
@@
   )
   (wire (pts (xy 181.61 95.25) (xy 203.2 95.25))
-    (stroke (width 0) (type default))
-  )
-  (wire (pts (xy 181.61 102.87) (xy 181.61 95.25))
     (stroke (width 0) (type default))
   )
@@
         )
       )
-    )
-  )
-  (symbol (lib_id "Connector:TestPoint") (at 181.61 102.87 270) (unit 1)
-    (in_bom yes) (on_board yes) (dnp no) (fields_autoplaced)
-    (property "Reference" "TP?" (at 186.69 101.6 90)
-      (effects (font (size 1.27 1.27)) (justify left))
-    )
-    (property "Value" "TestPoint" (at 186.69 104.14 90)
-      (effects (font (size 1.27 1.27)) (justify left))
-    )
-    (property "Footprint" "TestPoint:TestPoint_Pad_D2.0mm" (at 181.61 107.95 0)
-      (effects (font (size 1.27 1.27)) hide)
-    )
-    (property "Datasheet" "~" (at 181.61 107.95 0)
-      (effects (font (size 1.27 1.27)) hide)
-    )
-    (pin "1")
-    (instances
-      (project "ample"
-        (path "/bb5c9149-9eb8-4a9c-8d50-f58c12224ad5/00000000-0000-0000-0000-0000628f85ad"
-          (reference "TP?") (unit 1)
-        )
-        (path "/bb5c9149-9eb8-4a9c-8d50-f58c12224ad5/00000000-0000-0000-0000-0000628f8563"
-          (reference "TP?") (unit 1)
-        )
-        (path "/bb5c9149-9eb8-4a9c-8d50-f58c12224ad5/00000000-0000-0000-0000-0000628f83a4"
-          (reference "TP?") (unit 1)
-        )
-        (path "/bb5c9149-9eb8-4a9c-8d50-f58c12224ad5/00000000-0000-0000-0000-0000628f8ac6"
-          (reference "TP13") (unit 1)
-        )
-      )

Commit message: backport 1 for rev 00.01
Other:
- title: (none) -> ample/Input
Changed lines of the file:
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@@
 (kicad_sch (version 20230121) (generator eeschema)
   (paper "A4")
+  (title_block
+    (title "ample/Input")
+    (date "2023-07-14")
+    (rev "00.01")
+  )
   (junction (at 138.43 95.25) (diameter 0) (color 0 0 0 0)
   )
