File: src/hardware/pcb/ample/kicad/microcontroller.kicad_sch (KiCad schematic)
At the start: 13 parts, among them J4 Conn_02x03_Counter_Clockwise, J5 Conn_01x03, J6 Conn_01x03, J7 Conn_01x03, U10 ESP32-S2-WROVER

Commit message: rev 00.01 schematics almost done
Parts:
- removed C46: 10u, symbol Device:C_Small
- removed C47: 100n, symbol Device:C_Small
- removed MD1: ESP32-WROVER, Espressif_Systems-ESP32-WROVER-0-0-*, symbol ample-rescue:ESP32-WROVER-eec1
- removed U10: ESP32-S2-WROVER, RF_Module:ESP32-S2-WROVER, symbol RF_Module:ESP32-S2-WROVER
- added C27, C28: 100n, symbol Device:C_Small
- added C74, C75: 10u, symbol Device:C_Small
- added J8: Conn_01x03, symbol Connector_Generic:Conn_01x03
- added R36, R37, R38: 10k, symbol Device:R_Small
- added R39, R40: 0R, symbol Device:R_Small
- added R42, R43, R44, R45: np/100k, symbol Device:R_Small
- added SW1, SW2: SW_SPST, symbol Switch:SW_SPST
- added U14: ESP32-WROVER, LNIC_MCU:ESP32_WROVER_no_thermal_via, symbol LNIC_MCU:ESP32-WROVER
- C45: value 10u -> 100n
- D1: footprint (none) -> LED_SMD:LED_0603_1608Metric
- R26: value 10k -> 330R
- R27: value 10k -> 0R
Connections:
- net +3V3: now also R26.1, C28.1, C74.1, C75.1, J8.1 (Pin_1), R36.1, R38.1, R42.1, R43.1, R44.1, R45.1, U14.2 (3V3); no longer C45.1, R27.1
- net ESP32_BOOT: now also C45.1, R38.2, SW1.2 (B), U14.25 (IO0)
- net ESP32_EN: now also C27.1, R36.2, SW2.2 (B), U14.3 (EN); no longer R27.2
- net ESP32_RXD0: now also U14.34 (RXD0)
- net ESP32_TXD0: now also U14.35 (TXD0)
- net FILTER_SEL: now also R44.2, U14.8 (IO32)
- net F_SEL_0: now also R43.2, U14.6 (IO34)
- net F_SEL_1: now also R42.2, U14.7 (IO35)
- net GND: now also C27.2, C28.2, C74.2, C75.2, J8.3 (Pin_3), R37.2, SW1.1 (A), SW2.1 (A), U14.1 (GND), U14.15 (GND), U14.38 (GND), U14.39 (GND); no longer R26.2
- net SCL: now also U14.36 (IO22)
- net SDA: now also U14.33 (IO21)
- net LED_1: now reaches D1.1 (K)
- net LED_1: now also U14.31 (IO19)
- net at D1.2 (A): now also R26.2
- new net: R27.1, U14.30 (IO18)
- new net: R39.1, U14.29 (IO5)
- new net: R37.1, U14.14 (IO12)
- new net: R40.1, U14.23 (IO15)
- new net CODEC_INT: U14.37 (IO23)
- new net CODEC_nRST: U14.26 (IO4)
- new net CX_LRCK: R39.2
- new net CX_SCLK: R40.2
- new net CX_SDIN1: R27.2
- new net POT_SEL: J8.2 (Pin_2), R45.2, U14.9 (IO33)
- new net POT_VOLTAGE: U14.5 (SENSOR_VN)
- new net TOUCH_0: U14.10 (IO25)
- new net TOUCH_1: U14.11 (IO26)
- new net TOUCH_2: U14.12 (IO27)
- new net TOUCH_3: U14.13 (IO14)
- new net TOUCH_4: U14.16 (IO13)
- new net ~{MUTE}: U14.4 (SENSOR_VP)
- no-connect marks 9 -> 1
Other:
- note added: "maybe turn into external switch"
- note added: "select potentiometer as volume control or slider"
- moved on the sheet: D1, J4, J5, J6, J7

Commit message: finishing schematics
Parts:
- C78: renamed from C28; footprint (none) -> Capacitor_SMD:C_0603_1608Metric
- C79: renamed from C74; footprint (none) -> Capacitor_SMD:C_0603_1608Metric
- C80: renamed from C75; footprint (none) -> Capacitor_SMD:C_0603_1608Metric
- C81: renamed from C44; footprint (none) -> Capacitor_SMD:C_0603_1608Metric
- C82: renamed from C45; footprint (none) -> Capacitor_SMD:C_0603_1608Metric
- C83: renamed from C27; footprint (none) -> Capacitor_SMD:C_0603_1608Metric
- J4: footprint (none) -> Connector_PinHeader_2.54mm:PinHeader_2x03_P2.54mm_Vertical
- J5, J6, J7, J8: footprint (none) -> Connector_PinHeader_2.54mm:PinHeader_1x03_P2.54mm_Vertical
- R47: renamed from R37; footprint (none) -> Resistor_SMD:R_0603_1608Metric
- R48: renamed from R26; footprint (none) -> Resistor_SMD:R_0603_1608Metric
- R49: renamed from R27; footprint (none) -> Resistor_SMD:R_0603_1608Metric
- R50: renamed from R39; footprint (none) -> Resistor_SMD:R_0603_1608Metric
- R51: renamed from R40; footprint (none) -> Resistor_SMD:R_0603_1608Metric
- R52: renamed from R42; footprint (none) -> Resistor_SMD:R_0603_1608Metric
- R53: renamed from R43; footprint (none) -> Resistor_SMD:R_0603_1608Metric
- R54: renamed from R44; footprint (none) -> Resistor_SMD:R_0603_1608Metric
- R55: renamed from R45; footprint (none) -> Resistor_SMD:R_0603_1608Metric
- R56: renamed from R38; footprint (none) -> Resistor_SMD:R_0603_1608Metric
- R57: renamed from R36; footprint (none) -> Resistor_SMD:R_0603_1608Metric
- SW1, SW2: footprint (none) -> Button_Switch_THT:SW_PUSH_6mm
- renumbered D1 to D2, U14 to U11

Commit message: layout init
Parts:
- removed R52, R53, R54, R55: np/100k, Resistor_SMD:R_0603_1608Metric, symbol Device:R_Small
- removed SW1, SW2: SW_SPST, Button_Switch_THT:SW_PUSH_6mm, symbol Switch:SW_SPST
Connections:
- net TOUCH_2: no longer names the net of U11.12 (IO27)
- net TOUCH_3: no longer names the net of U11.13 (IO14)
- net TOUCH_4: no longer names the net of U11.16 (IO13)
- no-connect marks 1 -> 4

Commit message: rev 00.01
Parts:
- renumbered C78 to C86, C79 to C87, C80 to C88, C81 to C89, C82 to C90, C83 to C91, R47 to R41, R48 to R42, R49 to R43, R50 to R44, R51 to R45, R56 to R46, R57 to R47

Commit message: backport 1 for rev 00.01
Other:
- title: (none) -> ample/Microcontroller
Changed lines of the file:
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@@
 (kicad_sch (version 20230121) (generator eeschema)
   (paper "A4")
+  (title_block
+    (title "ample/Microcontroller")
+    (date "2023-07-14")
+    (rev "00.01")
+  )
   (junction (at 218.44 34.29) (diameter 0) (color 0 0 0 0)
   )
