File: src/hardware/pcb/ample/kicad/supply.kicad_sch (KiCad schematic)
At the start: 60 parts, among them J1 Jack-DC, J2 Conn_01x02, U12 LDL212DR, U13 RT7272A, U2 LDL212DR, U3 MAX660MX, U4 LDL212DR, U8 LDL212DR, U9 LP2951-3.0_SOIC

Commit message: rev 00.01 schematics almost done
Parts:
- removed C19, C52, C53: 10u, symbol Device:C_Small
- removed C21: 100n, symbol Device:C_Small
- removed R18: 10k, Resistor_SMD:R_0201_0603Metric, symbol Device:R_Small
- removed R33: 0R, Resistor_SMD:R_0201_0603Metric, symbol Device:R_Small
- removed R8: 91k, Resistor_SMD:R_0201_0603Metric, symbol Device:R_Small
- removed R9: 12k, Resistor_SMD:R_0201_0603Metric, symbol Device:R_Small
- removed U12: LDL212DR, Package_SO:SO-8_3.9x4.9mm_P1.27mm, symbol LNIC_Regulator_Linear:LDL212DR
Other:
- note removed: "R1 = 91, R2 = 12 V_out = 10.128 Error = 0.128 V_out_min = 9.681 V_out_max = 10.599 tol+ = 0.471 tol- = -0.447"
- moved on the sheet: C12, C14, C20, C22, C7, R11, R3, U3, U9

Commit message: finishing schematics
Parts:
- removed C8: 10u, symbol Device:C_Small
- removed FB1: Ferrite_Bead_Small, symbol ample-rescue:Ferrite_Bead_Small-Device
- removed J1: Jack-DC, symbol Connector:Jack-DC
- removed L1: 1u5, symbol Device:L_Small
- removed U9: LP2951-3.0_SOIC, Package_SO:SOIC-8_3.9x4.9mm_P1.27mm, symbol Regulator_Linear:LP2951-3.0_SOIC
- added C13, C25: 2u2, Capacitor_SMD:C_0603_1608Metric, symbol Device:C_Small
- added C18: 22n, Capacitor_SMD:C_0603_1608Metric, symbol Device:C_Small
- added C5: 220u, Capacitor_THT:CP_Radial_D6.3mm_P2.50mm, symbol Device:C_Polarized_Small
- added D?: LED_Small, LED_SMD:LED_0603_1608Metric, symbol Device:LED_Small
- added J1: DCJ200-05-A, LNIC_Connector_BarrelJack:DCJ200-05-A, symbol Connector:Barrel_Jack_Switch
- added L2: 104CDMCCDS-330MC, LNIC_Inductor_SMD:L_Sumida_104CDMCCDS, symbol Device:L_Small
- added R12, R16, R17, R18: 0R, Resistor_SMD:R_0603_1608Metric, symbol Device:R_Small
- added R21, R22: 10k, Resistor_SMD:R_0603_1608Metric, symbol Device:R_Small
- added R6: np/0R, Resistor_SMD:R_0603_1608Metric, symbol Device:R_Small
- added R?: 330R, Resistor_SMD:R_0603_1608Metric, symbol Device:R_Small
- added TP1, TP2, TP3, TP4, TP8 (x8): TestPoint, TestPoint:TestPoint_Pad_D2.0mm, symbol Connector:TestPoint
- added U5: LP2951-5.0_SOIC, Package_SO:SOIC-8_3.9x4.9mm_P1.27mm, symbol Regulator_Linear:LP2951-5.0_SOIC
- added np/R1: 18k, Resistor_SMD:R_0603_1608Metric, symbol Device:R_Small
- added np/R2: 56k, Resistor_SMD:R_0603_1608Metric, symbol Device:R_Small
- C1: renamed from C17; footprint (none) -> Capacitor_SMD:C_0603_1608Metric
- C10: renamed from C7; footprint (none) -> Capacitor_SMD:C_0603_1608Metric
- C11: renamed from C2; footprint (none) -> Capacitor_SMD:C_0603_1608Metric
- C12: renamed from C1; footprint (none) -> Capacitor_SMD:C_0603_1608Metric
- C14: footprint (none) -> Capacitor_SMD:C_0603_1608Metric
- C15: renamed from C5; footprint (none) -> Capacitor_SMD:C_0603_1608Metric
- C16: renamed from C4; footprint (none) -> Capacitor_SMD:C_0603_1608Metric
- C17: renamed from C20; footprint (none) -> Capacitor_SMD:C_0603_1608Metric
- C19: renamed from C50; footprint (none) -> Capacitor_SMD:C_0603_1608Metric
- C2: renamed from C16; footprint (none) -> Capacitor_SMD:C_0603_1608Metric
- C20: renamed from C51; footprint (none) -> Capacitor_SMD:C_0603_1608Metric
- C21: renamed from C11; footprint (none) -> Capacitor_SMD:C_0603_1608Metric
- C22: renamed from C48; footprint (none) -> Capacitor_SMD:C_0603_1608Metric
- C23: renamed from C49; footprint (none) -> Capacitor_SMD:C_0603_1608Metric
- C24: renamed from C3; footprint (none) -> Capacitor_SMD:C_0603_1608Metric
- C26: renamed from C6; footprint (none) -> Capacitor_SMD:C_0603_1608Metric
- C27: renamed from C13; footprint (none) -> Capacitor_SMD:C_0603_1608Metric
- C3: renamed from C18; footprint (none) -> Capacitor_SMD:C_0603_1608Metric
- C4: renamed from C22; footprint (none) -> Capacitor_SMD:C_0603_1608Metric
- C6: renamed from C9; footprint (none) -> Capacitor_SMD:C_0603_1608Metric
- C7: renamed from C12; footprint (none) -> Capacitor_SMD:C_0603_1608Metric
- C8: renamed from C10; footprint (none) -> Capacitor_SMD:C_0603_1608Metric
- C9: renamed from C15; footprint (none) -> Capacitor_SMD:C_0603_1608Metric
- J2: footprint (none) -> Connector_PinHeader_2.54mm:PinHeader_1x02_P2.54mm_Vertical
- L3: value 47u -> L_Eaton_HCM1A0805-470-R; footprint (none) -> LNIC_Inductor_SMD:L_Eaton_HCM1A0805
- R10: renamed from R1; footprint Resistor_SMD:R_0201_0603Metric -> Resistor_SMD:R_0603_1608Metric
- R11: renamed from R31; footprint Resistor_SMD:R_0201_0603Metric -> Resistor_SMD:R_0603_1608Metric
- R13: renamed from R30; footprint Resistor_SMD:R_0201_0603Metric -> Resistor_SMD:R_0603_1608Metric
- R14: renamed from R6; footprint Resistor_SMD:R_0201_0603Metric -> Resistor_SMD:R_0603_1608Metric
- R15: renamed from R7; footprint Resistor_SMD:R_0201_0603Metric -> Resistor_SMD:R_0603_1608Metric
- R19: renamed from R28; footprint Resistor_SMD:R_0201_0603Metric -> Resistor_SMD:R_0603_1608Metric
- R20: renamed from R29; footprint Resistor_SMD:R_0201_0603Metric -> Resistor_SMD:R_0603_1608Metric
- R23: renamed from R2; footprint Resistor_SMD:R_0201_0603Metric -> Resistor_SMD:R_0603_1608Metric
- R25: renamed from R10; footprint Resistor_SMD:R_0201_0603Metric -> Resistor_SMD:R_0603_1608Metric
- R26: renamed from R16; footprint Resistor_SMD:R_0201_0603Metric -> Resistor_SMD:R_0603_1608Metric
- R3: renamed from R13; footprint Resistor_SMD:R_0201_0603Metric -> Resistor_SMD:R_0603_1608Metric
- R4: renamed from R14; footprint Resistor_SMD:R_0201_0603Metric -> Resistor_SMD:R_0603_1608Metric
- R5: renamed from R15; footprint Resistor_SMD:R_0201_0603Metric -> Resistor_SMD:R_0603_1608Metric
- R7: renamed from R3; footprint Resistor_SMD:R_0201_0603Metric -> Resistor_SMD:R_0603_1608Metric
- R8: renamed from R11; footprint Resistor_SMD:R_0201_0603Metric -> Resistor_SMD:R_0603_1608Metric
- R9: renamed from R12; footprint Resistor_SMD:R_0201_0603Metric -> Resistor_SMD:R_0603_1608Metric
- renumbered U4 to U1, U3 to U2, U13 to U3, U8 to U4, U2 to U6
Connections:
- net +12V is gone; now on net VIN: C6.1
- net +3V3: now also TP8.1
- net +5V: now also R6.2, TP8.1; no longer C4.1, R7.1, U2.8 (V+)
- net +5V5: now also C25.1, R22.2, R?.1, TP3.1, TP8.1, U5.8 (IN)
- net +5VA: now also TP8.1
- net GND: now also C13.2, C25.2, C5.2, D?.1 (K), J1.2, J1.3, R21.1, TP8.1, TP8.1, TP8.1, TP8.1, np/R2.2
- net OP_VCC-: now also R18.1, TP2.1, np/R1.1
- net VIN: now also C5.1, J1.1, L2.1
- net at C12.1, C16.1, C8.1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: now also L2.2
- new net: R22.1, TP4.1, U5.5 (~{ERROR})
- new net: D?.2 (A), R?.2
- new net: C18.2, R16.1, U5.7 (FEEDBACK), np/R1.2, np/R2.1
- new net: C13.1, C4.1, R12.1, R6.1, R7.1, TP1.1, U2.8 (V+)
- new net: R21.2, U5.3 (SHUTDOWN)
- new net: C18.1, R12.2, R17.1, U5.1 (OUT)
- new net: R17.2, U5.2 (SENSE)
- new net: R16.2, U5.6 (VTAP)
- new net: R18.2, U5.4 (GND)
Other:
- note added: "R1"
- note added: "R1 = 56, R2 = 18 V_out = 5.077 Error = 0.077 V_out_min = 4.885 V_out_max = 5.279 tol+ = 0.202 tol- = -0.192"
- note added: "R2"
- note added: "fixed output regulator is untested use LP2951D (adjustable) if possible"
- note removed: "Maybe put an addtional (optional) negative rail regulator here"
- moved on the sheet: C1, C10, C11, C12, C14, C15, C16, C17, C19, C2, C20, C21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

Commit message: layout init
Parts:
- removed TP3: TestPoint, TestPoint:TestPoint_Pad_D2.0mm, symbol Connector:TestPoint
- added C100, C101, C105, C106, C107, C108, C33: np/10u, Capacitor_SMD:C_0603_1608Metric, symbol Device:C_Small
- added C104, C70: 10u, Capacitor_SMD:C_0603_1608Metric, symbol Device:C_Small
- R36: renamed from np/R1; value 18k -> np/18k
- R37: renamed from np/R2; value 56k -> np/56k
- U3: footprint Package_SO:SOIC-8-1EP_3.9x4.9mm_P1.27mm_EP2.41x3.3mm_ThermalVias -> Package_SO:SOIC-8-1EP_3.9x4.9mm_P1.27mm_EP2.41x3.3mm
Connections:
- net +3V3: now also C106.1
- net +5V: now also C105.1
- net +5V5: now also C101.1, C104.1, C107.1, C108.1
- net +5VA: now also C33.1
- net GND: now also C100.2, C101.2, C104.2, C105.2, C106.2, C107.2, C108.2, C33.2, C70.2
- net DCDC_IN: now reaches C12.1, C16.1, C8.1, L2.2, R9.1, U3.8 (VIN)
- net DCDC_IN: now also C100.1, C70.1
- net DCDC_SW: now reaches C19.1, L3.1, U3.1 (SW)
Other:
- note added: ">25V!"
- moved on the sheet: C12, C16, C5, C6, C8, C9, L2, R19, R20, R9

Commit message: rev 00.01
Parts:
- removed R12, R18, R7: 0R, Resistor_SMD:R_0603_1608Metric, symbol Device:R_Small
- removed R21: 10k, Resistor_SMD:R_0603_1608Metric, symbol Device:R_Small
- C10: renamed from C8; footprint Capacitor_SMD:C_0603_1608Metric -> Capacitor_SMD:C_0805_2012Metric
- C11: renamed from C70; footprint Capacitor_SMD:C_0603_1608Metric -> Capacitor_SMD:C_0805_2012Metric
- C8: renamed from C6; footprint Capacitor_SMD:C_0603_1608Metric -> Capacitor_SMD:C_0805_2012Metric
- renumbered C108 to C1, C104 to C12, C9 to C13, C100 to C14, C10 to C15, C11 to C16, C12 to C17, C13 to C18, C14 to C19, C1 to C2, C15 to C20, C16 to C21, C17 to C22, C18 to C23, C19 to C24, C20 to C25, C21 to C26, C22 to C27, C33 to C28, C23 to C29, C2 to C3, C101 to C30, C107 to C31, C24 to C32, C25 to C33, C26 to C34, C27 to C35, C106 to C36, C3 to C4, C4 to C6, C105 to C7, C7 to C9, L2 to L1, L3 to L2, R11 to R10, R13 to R11, R14 to R12, R15 to R13, R36 to R14, R37 to R15, R19 to R18, R20 to R19, R22 to R20, R23 to R21, R25 to R23, R26 to R24, R8 to R7, R9 to R8, R10 to R9, TP1 to TP3, TP2 to TP4, TP4 to TP9, TP8 to TP?
Connections:
- net GND: now also U5.3 (SHUTDOWN)
- net OP_VCC-: now also U5.4 (GND)
- net at U2.1 (FC): now also C18.1, C23.1, C6.1, R17.1, R6.1, TP3.1, U2.8 (V+), U5.1 (OUT)

Commit message: rev 00.01
Parts:
- removed TP3, TP9, TP? (x3): TestPoint, TestPoint:TestPoint_Pad_D2.0mm, symbol Connector:TestPoint

Commit message: backport 1 for rev 00.01
Other:
- title: (none) -> ample/Power Supply
Changed lines of the file:
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@@
   (paper "A3")
   (title_block
+    (title "ample/Power Supply")
+    (date "2023-07-14")
     (rev "00.01")
   )
