File: src/hardware/pcb/ample/kicad/ample.kicad_sch (KiCad schematic)
At the start: 2 parts

Commit message: rev 00.01 schematics almost done
Parts:
- R4, R5: value R_Small -> 4k7
Connections:
- net Microcontroller/SCL renamed Amplifier/SCL_1
- net Microcontroller/SDA renamed Amplifier/SDA_1
Other:
- sheet Output renamed DAC_Filter
- added sheet Control (Control.kicad_sch)
- sheet Amplifier ports: added FILT_LEFT_N, FILT_LEFT_P, FILT_RIGHT_N, FILT_RIGHT_P, MUTEC, SCL_1, SDA_1; removed none
- sheet Codec ports: added CODEC_INT, CODEC_nRST; removed CS42528_INT, CS42528_nRST, SAI_LRCLK, SAI_SCLK
- sheet DAC_Filter: file output.kicad_sch -> dac_filter.kicad_sch
- sheet DAC_Filter ports: added FILT_LEFT_N, FILT_LEFT_P, FILT_RIGHT_N, FILT_RIGHT_P; removed none
- sheet Microcontroller ports: added CODEC_INT, CODEC_nRST, CX_LRCK, CX_SCLK, CX_SDIN1, POT_VOLTAGE, TOUCH_0, TOUCH_1, TOUCH_2, TOUCH_3, TOUCH_4, ~{MUTE}; removed none
- moved on the sheet: R4, R5

Commit message: finishing schematics
Parts:
- added H1, H2, H3, H4: MountingHole, symbol Mechanical:MountingHole
- R1: renamed from R4; footprint (none) -> Resistor_SMD:R_0603_1608Metric
- R2: renamed from R5; footprint (none) -> Resistor_SMD:R_0603_1608Metric
Changed lines of the file:
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@@
   (symbol (lib_id "Device:R_Small") (at 151.13 107.95 0) (unit 1)
     (in_bom yes) (on_board yes) (dnp no)
-    (property "Reference" "R5" (at 152.6286 106.7816 0)
+    (property "Reference" "R2" (at 152.6286 106.7816 0)
       (effects (font (size 1.27 1.27)) (justify left))
     )
@@
       (effects (font (size 1.27 1.27)) (justify left))
     )
-    (property "Footprint" "" (at 151.13 107.95 0)
+    (property "Footprint" "Resistor_SMD:R_0603_1608Metric" (at 151.13 107.95 0)
       (effects (font (size 1.27 1.27)) hide)
     )
@@
       (project "ample"
         (path "/bb5c9149-9eb8-4a9c-8d50-f58c12224ad5"
-          (reference "R5") (unit 1)
+          (reference "R2") (unit 1)
         )
       )
@@
   (symbol (lib_id "Device:R_Small") (at 140.97 107.95 0) (unit 1)
     (in_bom yes) (on_board yes) (dnp no)
-    (property "Reference" "R4" (at 142.4686 106.7816 0)
+    (property "Reference" "R1" (at 142.4686 106.7816 0)
       (effects (font (size 1.27 1.27)) (justify left))
     )
@@
       (effects (font (size 1.27 1.27)) (justify left))
     )
-    (property "Footprint" "" (at 140.97 107.95 0)
+    (property "Footprint" "Resistor_SMD:R_0603_1608Metric" (at 140.97 107.95 0)
       (effects (font (size 1.27 1.27)) hide)
     )
@@
       (project "ample"
         (path "/bb5c9149-9eb8-4a9c-8d50-f58c12224ad5"
-          (reference "R4") (unit 1)
+          (reference "R1") (unit 1)
         )
       )
@@
   (symbol (lib_id "power:+3V3") (at 140.97 102.87 0) (unit 1)
     (in_bom yes) (on_board yes) (dnp no)
-    (property "Reference" "#PWR035" (at 140.97 106.68 0)
+    (property "Reference" "#PWR01" (at 140.97 106.68 0)
       (effects (font (size 1.27 1.27)) hide)
     )
@@
       (project "ample"
         (path "/bb5c9149-9eb8-4a9c-8d50-f58c12224ad5"
-          (reference "#PWR035") (unit 1)
+          (reference "#PWR01") (unit 1)
         )
       )
@@
   (symbol (lib_id "power:+3V3") (at 151.13 102.87 0) (unit 1)
     (in_bom yes) (on_board yes) (dnp no)
-    (property "Reference" "#PWR036" (at 151.13 106.68 0)
+    (property "Reference" "#PWR02" (at 151.13 106.68 0)
       (effects (font (size 1.27 1.27)) hide)
     )
@@
       (project "ample"
         (path "/bb5c9149-9eb8-4a9c-8d50-f58c12224ad5"
-          (reference "#PWR036") (unit 1)
+          (reference "#PWR02") (unit 1)
         )
       )
+    )
+  )
+  (symbol (lib_id "Mechanical:MountingHole") (at 25.4 176.53 0) (unit 1)
+    (in_bom yes) (on_board yes) (dnp no) (fields_autoplaced)
+    (property "Reference" "H2" (at 27.94 175.26 0)
+      (effects (font (size 1.27 1.27)) (justify left))
+    )
+    (property "Value" "MountingHole" (at 27.94 177.8 0)
+      (effects (font (size 1.27 1.27)) (justify left))
+    )
+    (property "Footprint" "" (at 25.4 176.53 0)
+      (effects (font (size 1.27 1.27)) hide)
+    )
+    (property "Datasheet" "~" (at 25.4 176.53 0)
+      (effects (font (size 1.27 1.27)) hide)
+    )
+    (instances
+      (project "ample"
+        (path "/bb5c9149-9eb8-4a9c-8d50-f58c12224ad5"
+          (reference "H2") (unit 1)
+        )
+      )
+    )
+  )
+  (symbol (lib_id "Mechanical:MountingHole") (at 25.4 182.88 0) (unit 1)
+    (in_bom yes) (on_board yes) (dnp no) (fields_autoplaced)
+    (property "Reference" "H3" (at 27.94 181.61 0)
+      (effects (font (size 1.27 1.27)) (justify left))
+    )
+    (property "Value" "MountingHole" (at 27.94 184.15 0)
+      (effects (font (size 1.27 1.27)) (justify left))
+    )
+    (property "Footprint" "" (at 25.4 182.88 0)
+      (effects (font (size 1.27 1.27)) hide)
+    )
+    (property "Datasheet" "~" (at 25.4 182.88 0)
+      (effects (font (size 1.27 1.27)) hide)
+    )
+    (instances
+      (project "ample"
+        (path "/bb5c9149-9eb8-4a9c-8d50-f58c12224ad5"
+          (reference "H3") (unit 1)
+        )
+      )
+    )
+  )
+  (symbol (lib_id "Mechanical:MountingHole") (at 25.4 189.23 0) (unit 1)
+    (in_bom yes) (on_board yes) (dnp no) (fields_autoplaced)
+    (property "Reference" "H4" (at 27.94 187.96 0)
+      (effects (font (size 1.27 1.27)) (justify left))
+    )
+    (property "Value" "MountingHole" (at 27.94 190.5 0)
+      (effects (font (size 1.27 1.27)) (justify left))
+    )
+    (property "Footprint" "" (at 25.4 189.23 0)
+      (effects (font (size 1.27 1.27)) hide)
+    )
+    (property "Datasheet" "~" (at 25.4 189.23 0)
+      (effects (font (size 1.27 1.27)) hide)
+    )
+    (instances
+      (project "ample"
+        (path "/bb5c9149-9eb8-4a9c-8d50-f58c12224ad5"
+          (reference "H4") (unit 1)
+        )
+      )
+    )
+  )
+  (symbol (lib_id "Mechanical:MountingHole") (at 25.4 170.18 0) (unit 1)
+    (in_bom yes) (on_board yes) (dnp no) (fields_autoplaced)
+    (property "Reference" "H1" (at 27.94 168.91 0)
+      (effects (font (size 1.27 1.27)) (justify left))
+    )
+    (property "Value" "MountingHole" (at 27.94 171.45 0)
+      (effects (font (size 1.27 1.27)) (justify left))
+    )
+    (property "Footprint" "" (at 25.4 170.18 0)
+      (effects (font (size 1.27 1.27)) hide)
+    )
+    (property "Datasheet" "~" (at 25.4 170.18 0)
+      (effects (font (size 1.27 1.27)) hide)
+    )
+    (instances
+      (project "ample"
+        (path "/bb5c9149-9eb8-4a9c-8d50-f58c12224ad5"
+          (reference "H1") (unit 1)
+        )
+      )

Commit message: layout init
Parts:
- H1, H2, H3, H4: footprint (none) -> MountingHole:MountingHole_3.2mm_M3
Other:
- sheet Codec ports: added AOUTA+, AOUTA-, AOUTB+, AOUTB-; removed AOUTA1+, AOUTA1-, AOUTB1+, AOUTB1-
- sheet Control ports: added none; removed TOUCH_2, TOUCH_3, TOUCH_4
- sheet DAC_Filter ports: added AOUTA+, AOUTA-, AOUTB+, AOUTB-; removed AOUTA1+, AOUTA1-, AOUTB1+, AOUTB1-
- sheet Microcontroller ports: added none; removed TOUCH_2, TOUCH_3, TOUCH_4
Changed lines of the file:
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@@
-    (stroke (width 0) (type default))
-  )
-  (wire (pts (xy 205.74 116.84) (xy 222.25 116.84))
     (stroke (width 0) (type default))
   )
@@
     (stroke (width 0) (type default))
   )
-  (wire (pts (xy 205.74 114.3) (xy 222.25 114.3))
-    (stroke (width 0) (type default))
-  )
   (wire (pts (xy 151.13 116.84) (xy 166.37 116.84))
     (stroke (width 0) (type default))
@@
   )
   (wire (pts (xy 115.57 135.89) (xy 176.53 135.89))
-    (stroke (width 0) (type default))
-  )
-  (wire (pts (xy 205.74 119.38) (xy 222.25 119.38))
     (stroke (width 0) (type default))
   )
@@
     )
   )
+  (symbol (lib_id "Mechanical:MountingHole") (at 25.4 189.23 0) (unit 1)
+    (in_bom yes) (on_board yes) (dnp no) (fields_autoplaced)
+    (property "Reference" "H4" (at 27.94 187.96 0)
+      (effects (font (size 1.27 1.27)) (justify left))
+    )
+    (property "Value" "MountingHole" (at 27.94 190.5 0)
+      (effects (font (size 1.27 1.27)) (justify left))
+    )
+    (property "Footprint" "MountingHole:MountingHole_3.2mm_M3" (at 25.4 189.23 0)
+      (effects (font (size 1.27 1.27)) hide)
+    )
+    (property "Datasheet" "~" (at 25.4 189.23 0)
+      (effects (font (size 1.27 1.27)) hide)
+    )
+    (instances
+      (project "ample"
+        (path "/bb5c9149-9eb8-4a9c-8d50-f58c12224ad5"
+          (reference "H4") (unit 1)
+        )
+      )
+    )
+  )
+  (symbol (lib_id "Mechanical:MountingHole") (at 25.4 170.18 0) (unit 1)
+    (in_bom yes) (on_board yes) (dnp no) (fields_autoplaced)
+    (property "Reference" "H1" (at 27.94 168.91 0)
+      (effects (font (size 1.27 1.27)) (justify left))
+    )
+    (property "Value" "MountingHole" (at 27.94 171.45 0)
+      (effects (font (size 1.27 1.27)) (justify left))
+    )
+    (property "Footprint" "MountingHole:MountingHole_3.2mm_M3" (at 25.4 170.18 0)
+      (effects (font (size 1.27 1.27)) hide)
+    )
+    (property "Datasheet" "~" (at 25.4 170.18 0)
+      (effects (font (size 1.27 1.27)) hide)
+    )
+    (instances
+      (project "ample"
+        (path "/bb5c9149-9eb8-4a9c-8d50-f58c12224ad5"
+          (reference "H1") (unit 1)
+        )
+      )
+    )
+  )
+  (symbol (lib_id "Mechanical:MountingHole") (at 25.4 182.88 0) (unit 1)
+    (in_bom yes) (on_board yes) (dnp no) (fields_autoplaced)
+    (property "Reference" "H3" (at 27.94 181.61 0)
+      (effects (font (size 1.27 1.27)) (justify left))
+    )
+    (property "Value" "MountingHole" (at 27.94 184.15 0)
+      (effects (font (size 1.27 1.27)) (justify left))
+    )
+    (property "Footprint" "MountingHole:MountingHole_3.2mm_M3" (at 25.4 182.88 0)
+      (effects (font (size 1.27 1.27)) hide)
+    )
+    (property "Datasheet" "~" (at 25.4 182.88 0)
+      (effects (font (size 1.27 1.27)) hide)
+    )
+    (instances
+      (project "ample"
+        (path "/bb5c9149-9eb8-4a9c-8d50-f58c12224ad5"
+          (reference "H3") (unit 1)
+        )
+      )
+    )
+  )
   (symbol (lib_id "Mechanical:MountingHole") (at 25.4 176.53 0) (unit 1)
     (in_bom yes) (on_board yes) (dnp no) (fields_autoplaced)
@@
       (effects (font (size 1.27 1.27)) (justify left))
     )
-    (property "Footprint" "" (at 25.4 176.53 0)
+    (property "Footprint" "MountingHole:MountingHole_3.2mm_M3" (at 25.4 176.53 0)
       (effects (font (size 1.27 1.27)) hide)
     )
@@
         (path "/bb5c9149-9eb8-4a9c-8d50-f58c12224ad5"
           (reference "H2") (unit 1)
-        )
-      )
-    )
-  )
-  (symbol (lib_id "Mechanical:MountingHole") (at 25.4 182.88 0) (unit 1)
-    (in_bom yes) (on_board yes) (dnp no) (fields_autoplaced)
-    (property "Reference" "H3" (at 27.94 181.61 0)
-      (effects (font (size 1.27 1.27)) (justify left))
-    )
-    (property "Value" "MountingHole" (at 27.94 184.15 0)
-      (effects (font (size 1.27 1.27)) (justify left))
-    )
-    (property "Footprint" "" (at 25.4 182.88 0)
-      (effects (font (size 1.27 1.27)) hide)
-    )
-    (property "Datasheet" "~" (at 25.4 182.88 0)
-      (effects (font (size 1.27 1.27)) hide)
-    )
-    (instances
-      (project "ample"
-        (path "/bb5c9149-9eb8-4a9c-8d50-f58c12224ad5"
-          (reference "H3") (unit 1)
-        )
-      )
-    )
-  )
-  (symbol (lib_id "Mechanical:MountingHole") (at 25.4 189.23 0) (unit 1)
-    (in_bom yes) (on_board yes) (dnp no) (fields_autoplaced)
-    (property "Reference" "H4" (at 27.94 187.96 0)
-      (effects (font (size 1.27 1.27)) (justify left))
-    )
-    (property "Value" "MountingHole" (at 27.94 190.5 0)
-      (effects (font (size 1.27 1.27)) (justify left))
-    )
-    (property "Footprint" "" (at 25.4 189.23 0)
-      (effects (font (size 1.27 1.27)) hide)
-    )
-    (property "Datasheet" "~" (at 25.4 189.23 0)
-      (effects (font (size 1.27 1.27)) hide)
-    )
-    (instances
-      (project "ample"
-        (path "/bb5c9149-9eb8-4a9c-8d50-f58c12224ad5"
-          (reference "H4") (unit 1)
-        )
-      )
-    )
-  )
-  (symbol (lib_id "Mechanical:MountingHole") (at 25.4 170.18 0) (unit 1)
-    (in_bom yes) (on_board yes) (dnp no) (fields_autoplaced)
-    (property "Reference" "H1" (at 27.94 168.91 0)
-      (effects (font (size 1.27 1.27)) (justify left))
-    )
-    (property "Value" "MountingHole" (at 27.94 171.45 0)
-      (effects (font (size 1.27 1.27)) (justify left))
-    )
-    (property "Footprint" "" (at 25.4 170.18 0)
-      (effects (font (size 1.27 1.27)) hide)
-    )
-    (property "Datasheet" "~" (at 25.4 170.18 0)
-      (effects (font (size 1.27 1.27)) hide)
-    )
-    (instances
-      (project "ample"
-        (path "/bb5c9149-9eb8-4a9c-8d50-f58c12224ad5"
-          (reference "H1") (unit 1)
         )
       )
@@
       (effects (font (size 1.27 1.27)) (justify left))
     )
-    (pin "TOUCH_4" output (at 205.74 114.3 0)
-      (effects (font (size 1.27 1.27)) (justify right))
-    )
     (pin "TOUCH_1" output (at 205.74 121.92 0)
       (effects (font (size 1.27 1.27)) (justify right))
     )
     (pin "TOUCH_0" output (at 205.74 124.46 0)
-      (effects (font (size 1.27 1.27)) (justify right))
-    )
-    (pin "TOUCH_2" output (at 205.74 119.38 0)
-      (effects (font (size 1.27 1.27)) (justify right))
-    )
-    (pin "TOUCH_3" output (at 205.74 116.84 0)
       (effects (font (size 1.27 1.27)) (justify right))
     )
@@
       (effects (font (size 1.27 1.27)) (justify left))
     )
-    (pin "AOUTA1-" output (at 115.57 74.93 0)
-      (effects (font (size 1.27 1.27)) (justify right))
-    )
-    (pin "AOUTA1+" output (at 115.57 72.39 0)
-      (effects (font (size 1.27 1.27)) (justify right))
-    )
-    (pin "AOUTB1+" output (at 115.57 77.47 0)
-      (effects (font (size 1.27 1.27)) (justify right))
-    )
-    (pin "AOUTB1-" output (at 115.57 80.01 0)
+    (pin "AOUTA-" output (at 115.57 74.93 0)
+      (effects (font (size 1.27 1.27)) (justify right))
+    )
+    (pin "AOUTA+" output (at 115.57 72.39 0)
+      (effects (font (size 1.27 1.27)) (justify right))
+    )
+    (pin "AOUTB+" output (at 115.57 77.47 0)
+      (effects (font (size 1.27 1.27)) (justify right))
+    )
+    (pin "AOUTB-" output (at 115.57 80.01 0)
       (effects (font (size 1.27 1.27)) (justify right))
     )
@@
       (effects (font (size 1.27 1.27)) (justify left))
     )
-    (pin "TOUCH_2" input (at 222.25 119.38 180)
-      (effects (font (size 1.27 1.27)) (justify left))
-    )
-    (pin "TOUCH_3" input (at 222.25 116.84 180)
-      (effects (font (size 1.27 1.27)) (justify left))
-    )
-    (pin "TOUCH_4" input (at 222.25 114.3 180)
-      (effects (font (size 1.27 1.27)) (justify left))
-    )
     (instances
       (project "ample"
@@
       (effects (font (size 1.27 1.27)) (justify left top))
     )
-    (pin "AOUTA1-" input (at 130.81 74.93 180)
-      (effects (font (size 1.27 1.27)) (justify left))
-    )
-    (pin "AOUTA1+" input (at 130.81 72.39 180)
-      (effects (font (size 1.27 1.27)) (justify left))
-    )
-    (pin "AOUTB1+" input (at 130.81 77.47 180)
-      (effects (font (size 1.27 1.27)) (justify left))
-    )
-    (pin "AOUTB1-" input (at 130.81 80.01 180)
-      (effects (font (size 1.27 1.27)) (justify left))
-    )
+    (pin "AOUTA-" input (at 130.81 74.93 180)
+      (effects (font (size 1.27 1.27)) (justify left))
+    )
+    (pin "AOUTA+" input (at 130.81 72.39 180)
+      (effects (font (size 1.27 1.27)) (justify left))
+    )
+    (pin "AOUTB+" input (at 130.81 77.47 180)
+      (effects (font (size 1.27 1.27)) (justify left))
+    )
+    (pin "AOUTB-" input (at 130.81 80.01 180)
+      (effects (font (size 1.27 1.27)) (justify left))
+    )

Commit message: rev 00.01
Changed lines of the file:
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@@
+    )
+  )
+  (symbol (lib_id "Graphic:Logo_Open_Hardware_Small") (at 53.34 186.69 0) (unit 1)
+    (in_bom no) (on_board no) (dnp no) (fields_autoplaced)
+    (property "Reference" "#SYM1" (at 53.34 179.705 0)
+      (effects (font (size 1.27 1.27)) hide)
+    )
+    (property "Value" "Logo_Open_Hardware_Small" (at 53.34 192.405 0)
+      (effects (font (size 1.27 1.27)) hide)
+    )
+    (property "Footprint" "Symbol:OSHW-Symbol_33.5x30mm_SilkScreen" (at 53.34 186.69 0)
+      (effects (font (size 1.27 1.27)) hide)
+    )
+    (property "Datasheet" "~" (at 53.34 186.69 0)
+      (effects (font (size 1.27 1.27)) hide)
+    )
+    (property "Sim.Enable" "0" (at 53.34 186.69 0)
+      (effects (font (size 1.27 1.27)) hide)
+    )
+    (instances
+      (project "ample"
+        (path "/bb5c9149-9eb8-4a9c-8d50-f58c12224ad5"
+          (reference "#SYM1") (unit 1)
+        )
+      )
     )
   )

Commit message: backport 1 for rev 00.01
Other:
- title: (none) -> Ample/Hierarchy
Changed lines of the file:
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@@
 (kicad_sch (version 20230121) (generator eeschema)
   (paper "A4")
+  (title_block
+    (title "Ample/Hierarchy")
+    (date "2023-07-14")
+    (rev "00.01")
+  )
   (junction (at 166.37 116.84) (diameter 0) (color 0 0 0 0)
   )

Commit message: change sheet name
Other:
- title: Ample/Hierarchy -> ample/Hierarchy
Changed lines of the file:
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@@
   (paper "A4")
   (title_block
-    (title "Ample/Hierarchy")
+    (title "ample/Hierarchy")
     (date "2023-07-14")
     (rev "00.01")
